File: ASISTE.kicad_pcb (KiCad board)
At the start: 4 copper layers, 33.1 x 20.3 mm, 70 parts, among them IC1 MAX30105, J1 USB_B_Micro_SMD, J2 Conn_01x02, Q1 NTK3134NT1G, Q2 NTK3134NT1G, Q3 NTK3134NT1G, Q4 DMP1045U, SW1 SW_SPST, U1 MCP73831, U2 XC6415CC91MR-G, U3 MPU-6050, U4 TMP112AIDRLR, U5 nRF51x22-QFxx, Y1 Crystal_GND24_2520, Y2 Crystal_3.2x1.5

Commit message: Actualizando
Parts:
- removed the C1 at (170.1, 119.2)
- removed the C12 at (166.6, 119.7)
- added C11: C_0402_100nF, ASISTE:C_0402, F.Cu at (166.6, 119.7)
- R4: moved to F.Cu
- moved PROG1 12.0 mm to (159.3, 121.7), turned to 0 degrees
- moved D1 9.12 mm to (169.9, 119.0), turned to 90 degrees
- moved R3 8.14 mm to (167.5, 119.6), turned to 180 degrees
- moved SW1 7.84 mm to (169.9, 113.3), turned to 270 degrees
- moved R4 6.72 mm to (169.9, 113.3), turned to 270 degrees
- moved R2 6.61 mm to (167.5, 118.3), turned to 180 degrees
- moved R1 5.31 mm to (167.5, 117.0), turned to 180 degrees
- moved R12 0.90 mm to (156.7, 120.4)
- moved R13 0.77 mm to (156.7, 119.2)
- moved U3 0.64 mm to (161.8, 119.3)
- moved C12 0.52 mm to (156.7, 118.0)
- moved C21 0.51 mm to (156.1, 116.3)
- renumbered C2 to C1, C11 to C10, C13 to C12, C14 to C13, C15 to C14, C16 to C15, C17 to C16, C18 to C17, C19 to C18, C20 to C19, C3 to C2, C21 to C20, C22 to C21, C23 to C22, C24 to C23, C25 to C24, C26 to C25, C27 to C26, C28 to C27, C4 to C3, C5 to C4, C6 to C5, C7 to C6, C8 to C7, C9 to C8, C10 to C9
Connections:
- net /micro/MPU_PROG_RX renamed /micro/MCU_PROG_RX
Routing:
- net /micro/MCU_PROG_TX: track 0.00 -> 9.78 mm, vias 0 -> 1
- net /micro/MCU_PROG_RX: track 0.00 -> 9.45 mm, vias 0 -> 1
- net /micro/MCU_DEBUG_SWDIO: track 0.00 -> 9.37 mm, vias 0 -> 1
- net /micro/MCU_DEBUG_SWCLK: track 0.00 -> 7.73 mm, vias 0 -> 1
- net +3V3: track 41.7 -> 38.0 mm, vias 12 -> 14
- net /micro/LED_RED: track 6.29 -> 9.18 mm
- net GND: track 90.9 -> 88.6 mm, vias 34 -> 31
- net /imu/IMU_SDA: track 11.2 -> 9.39 mm
- net /micro/BUTTON: track 15.0 -> 13.6 mm, vias 1 -> 2
- net /micro/LED_GREEN: track 6.99 -> 8.40 mm
- net /micro/LED_BLUE: track 6.92 -> 7.63 mm
- net /imu/IMU_INT: track 10.9 -> 11.4 mm
