File: ASISTE.sch (KiCad schematic (older format))
At the start: 4 parts

Commit message: Terminado esquemático. Falta revisar
Parts:
- added C?: C_0603_1uF, ASISTE:C_0603, symbol Asiste:C_0603_1uF
- added PROG?: SMD_01x06, ASISTE:SMD_PROG, symbol Asiste:SMD_01x06
- added R?: R_0402_100, ASISTE:R_0402, symbol Asiste:R_0402_100
- added SW?: SW_SPST, ASISTE:SW_SPST_PTS810, symbol Asiste:SW_SPST
Connections:
- net labels added: GND, VCC
- wire segments 26 -> 48
Changed lines of the file:
@@
 $EndSheet
 $Sheet
-S 2750 4200 1400 650
+S 2750 4300 1400 500
 U 5B56C12F
 F0 "power" 60
 F1 "power.sch" 60
-F2 "BAT_CHG_STAT" O R 4150 4400 60
+F2 "BAT_CHG_STAT" O R 4150 4550 60
 F3 "BAT_SENSE" O R 4150 4650 60
+F4 "PWR_EN" I R 4150 4450 60
 $EndSheet
 $Sheet
@@
 F3 "MCU_SCL2" O R 7200 4750 60
 F4 "MCU_INT2" I R 7200 4550 60
-F5 "MPU_PROG_RX" I L 5250 3350 60
-F6 "MCU_PROG_TX" I L 5250 3450 60
+F5 "MPU_PROG_RX" I L 5250 3250 60
+F6 "MCU_PROG_TX" I L 5250 3150 60
 F7 "MPU_SDA1" B R 7200 3250 60
 F8 "MPU_INT1" I R 7200 3150 60
 F9 "MCU_AN1" I L 5250 4650 60
-F10 "MCU_DEBUG_SWCLK" I L 5250 3150 60
-F11 "MCU_DEBUG_SWDIO" I L 5250 3250 60
+F10 "MCU_DEBUG_SWCLK" I L 5250 3350 60
+F11 "MCU_DEBUG_SWDIO" I L 5250 3450 60
 F12 "MPU_SCL1" O R 7200 3350 60
 F13 "MCU_INT3" I R 7200 4050 60
@@
 F15 "LED_RED" O L 5250 3750 60
 F16 "LED_BLUE" O L 5250 3950 60
+F17 "PWR_EN" O L 5250 4450 60
+F18 "BAT_CHG_STAT" I L 5250 4550 60
+F19 "BUTTON" I L 5250 3650 60
 $EndSheet
 Wire Wire Line
@@
 $EndComp
 Wire Wire Line
-	2500 2550 2500 2650
+	2500 2550 2500 2600
 $Comp
 L Asiste:+3V3 #PWR?
@@
 Wire Wire Line
 	2850 3050 2850 3150
+Wire Wire Line
+	5250 4450 4150 4450
+Wire Wire Line
+	5250 4550 4150 4550
+$Comp
+L Asiste:SMD_01x06 PROG?
+U 1 1 5B936A3E
+P 4200 3150
+F 0 "PROG?" H 4300 3500 50  0000 C CNN
+F 1 "SMD_01x06" H 4200 2750 50  0001 C CNN
+F 2 "ASISTE:SMD_PROG" H 4100 3350 50  0001 C CNN
+F 3 "~" H 4200 3150 50  0001 C CNN
+	1    4200 3150
+	1    0    0    -1
+$EndComp
+Wire Wire Line
+	4400 3150 5250 3150
+Wire Wire Line
+	4400 3250 5250 3250
+Wire Wire Line
+	4400 3350 5250 3350
+Wire Wire Line
+	4400 3450 5250 3450
+Wire Wire Line
+	4400 2950 4500 2950
+$Comp
+L Asiste:GND #PWR?
+U 1 1 5B9387C2
+P 4800 3050
+F 0 "#PWR?" H 4800 2800 50  0001 C CNN
+F 1 "GND" V 4805 2922 50  0000 R CNN
+F 2 "" H 4800 3050 50  0001 C CNN
+F 3 "" H 4800 3050 50  0001 C CNN
+	1    4800 3050
+	0    -1   -1   0
+$EndComp
+Wire Wire Line
+	4400 3050 4700 3050
+$Comp
+L Asiste:C_0603_1uF C?
+U 1 1 5B93A003
+P 4700 2850
+F 0 "C?" H 4815 2896 50  0000 L CNN
+F 1 "C_0603_1uF" H 4500 2300 50  0001 L CNN
+F 2 "ASISTE:C_0603" H 4750 2600 50  0001 C CNN
+F 3 "https://www.mouser.es/datasheet/2/396/mlcc02_e-1307760.pdf" H 5250 2500 50  0001 C CNN
+F 4 "LMK107B7105KAHT" H 4700 2400 60  0001 C CNN "man#"
+F 5 "1uF" H 4815 2805 50  0000 L CNN "Capacitance"
+F 6 "10V" H 4700 2400 60  0001 C CNN "Voltage"
+	1    4700 2850
+	1    0    0    -1
+$EndComp
+Wire Wire Line
+	4500 2600 4500 2950
+Wire Wire Line
+	4700 2700 4700 2600
+Wire Wire Line
+	4500 2600 4700 2600
+Wire Wire Line
+	4700 3000 4700 3050
+Connection ~ 4700 3050
+Wire Wire Line
+	4700 3050 4800 3050
+$Comp
+L Asiste:SW_SPST SW?
+U 1 1 5B897F2A
+P 3350 3300
+F 0 "SW?" V 3304 3398 50  0000 L CNN
+F 1 "SW_SPST" V 3395 3398 50  0000 L CNN
+F 2 "ASISTE:SW_SPST_PTS810" H 3400 3100 50  0001 C CNN
+F 3 "https://www.mouser.es/datasheet/2/60/pts810-1382876.pdf" H 3300 3000 50  0001 C CNN
+F 4 "PTS810SJK250SMTRLFS" H 3350 2900 60  0001 C CNN "man#"
+	1    3350 3300
+	0    1    1    0
+$EndComp
+$Comp
+L Asiste:R_0402_100 R?
+U 1 1 5B89881E
+P 3350 2850
+F 0 "R?" H 3420 2896 50  0000 L CNN
+F 1 "R_0402_100" H 3350 2300 50  0001 C CNN
+F 2 "ASISTE:R_0402" H 3350 2400 50  0001 C CNN
+F 3 "https://www.mouser.es/datasheet/2/315/AOA0000C334-1314047.pdf" H 3350 2500 50  0001 C CNN
+F 4 "ERJ-U02D1000X" H 3300 2600 60  0001 C CNN "man#"
+F 5 "100" H 3420 2805 50  0000 L CNN "Resistance"
+	1    3350 2850
+	1    0    0    -1
+$EndComp
+Wire Wire Line
+	3350 2700 3350 2600
+Wire Wire Line
+	3350 2600 2500 2600
+Connection ~ 2500 2600
+Wire Wire Line
+	2500 2600 2500 2650
+Connection ~ 4700 2600
+$Comp
+L Asiste:VCC #PWR?
+U 1 1 5B93814B
+P 4700 2600
+F 0 "#PWR?" H 4700 2450 50  0001 C CNN
+F 1 "VCC" H 4715 2773 50  0000 C CNN
+F 2 "" H 4700 2600 50  0001 C CNN
+F 3 "" H 4700 2600 50  0001 C CNN
+	1    4700 2600
+	1    0    0    -1
+$EndComp
+Wire Wire Line
+	3350 3000 3350 3050
+$Comp
+L Asiste:GND #PWR?
+U 1 1 5B89A405
+P 3350 3600
+F 0 "#PWR?" H 3350 3350 50  0001 C CNN
+F 1 "GND" H 3200 3550 50  0000 C CNN
+F 2 "" H 3350 3600 50  0001 C CNN
+F 3 "" H 3350 3600 50  0001 C CNN
+	1    3350 3600
+	1    0    0    -1
+$EndComp
+Wire Wire Line
+	3350 3500 3350 3600
+Wire Wire Line
+	5250 3650 3850 3650
+Wire Wire Line
+	3850 3650 3850 3050
+Wire Wire Line
+	3850 3050 3350 3050
+Connection ~ 3350 3050
+Wire Wire Line
+	3350 3050 3350 3100
 $EndSCHEMATC

Commit message: Esquemático parcialmente revisado. Falta revisar pines y correspondencia con footprints
Parts:
- gave numbers to parts that had none: 8
Changed lines of the file:
@@
 F4 "IMU_SCL" I L 8250 3350 60
-$EndSheet
-$Sheet
-S 5250 3000 1950 1850
-U 5B56C637
-F0 "micro" 60
-F1 "micro.sch" 60
-F2 "MCU_SDA2" B R 7200 4650 60
-F3 "MCU_SCL2" O R 7200 4750 60
-F4 "MCU_INT2" I R 7200 4550 60
-F5 "MPU_PROG_RX" I L 5250 3250 60
-F6 "MCU_PROG_TX" I L 5250 3150 60
-F7 "MPU_SDA1" B R 7200 3250 60
-F8 "MPU_INT1" I R 7200 3150 60
-F9 "MCU_AN1" I L 5250 4650 60
-F10 "MCU_DEBUG_SWCLK" I L 5250 3350 60
-F11 "MCU_DEBUG_SWDIO" I L 5250 3450 60
-F12 "MPU_SCL1" O R 7200 3350 60
-F13 "MCU_INT3" I R 7200 4050 60
-F14 "LED_GREEN" O L 5250 3850 60
-F15 "LED_RED" O L 5250 3750 60
-F16 "LED_BLUE" O L 5250 3950 60
-F17 "PWR_EN" O L 5250 4450 60
-F18 "BAT_CHG_STAT" I L 5250 4550 60
-F19 "BUTTON" I L 5250 3650 60
 $EndSheet
 Wire Wire Line
@@
 	7550 3250 8250 3250
 $Comp
-L Asiste:LED_ARGB D?
+L Asiste:LED_ARGB D101
 U 1 1 5B7F5EAD
 P 2500 2850
-F 0 "D?" H 2500 2383 50  0000 C CNN
+F 0 "D101" H 2500 2383 50  0000 C CNN
 F 1 "LED_ARGB" H 2500 2474 50  0000 C CNN
 F 2 "ASISTE:LED_Cree-PLCC4_2x2mm_CW" H 2500 2250 50  0001 C CNN
@@
 	2500 2550 2500 2600
 $Comp
-L Asiste:+3V3 #PWR?
+L Asiste:+3V3 #PWR0101
 U 1 1 5B7F63F5
 P 2500 2550
-F 0 "#PWR?" H 2500 2400 50  0001 C CNN
+F 0 "#PWR0101" H 2500 2400 50  0001 C CNN
 F 1 "+3V3" H 2515 2723 50  0000 C CNN
 F 2 "" H 2500 2550 50  0001 C CNN
@@
 $EndComp
 $Comp
-L Asiste:R_0402_100 R?
+L Asiste:R_0402_100 R103
 U 1 1 5B787251
 P 2850 3300
-F 0 "R?" H 2920 3346 50  0000 L CNN
+F 0 "R103" H 2920 3346 50  0000 L CNN
 F 1 "R_0402_100" H 2850 2750 50  0001 C CNN
 F 2 "ASISTE:R_0402" H 2850 2850 50  0001 C CNN
@@
 $EndComp
 $Comp
-L Asiste:R_0402_33 R?
+L Asiste:R_0402_33 R102
 U 1 1 5B78744C
 P 2500 3300
-F 0 "R?" H 2570 3346 50  0000 L CNN
+F 0 "R102" H 2570 3346 50  0000 L CNN
 F 1 "R_0402_33" H 2500 2750 50  0001 C CNN
 F 2 "ASISTE:R_0402" H 2500 2850 50  0001 C CNN
@@
 $EndComp
 $Comp
-L Asiste:R_0402_33 R?
+L Asiste:R_0402_33 R101
 U 1 1 5B7874B2
 P 2150 3300
-F 0 "R?" H 2220 3346 50  0000 L CNN
+F 0 "R101" H 2220 3346 50  0000 L CNN
 F 1 "R_0402_33" H 2150 2750 50  0001 C CNN
 F 2 "ASISTE:R_0402" H 2150 2850 50  0001 C CNN
@@
 	5250 4550 4150 4550
 $Comp
-L Asiste:SMD_01x06 PROG?
+L Asiste:SMD_01x06 PROG101
 U 1 1 5B936A3E
 P 4200 3150
-F 0 "PROG?" H 4300 3500 50  0000 C CNN
+F 0 "PROG101" H 4300 3500 50  0000 C CNN
 F 1 "SMD_01x06" H 4200 2750 50  0001 C CNN
 F 2 "ASISTE:SMD_PROG" H 4100 3350 50  0001 C CNN
@@
 	4400 2950 4500 2950
 $Comp
-L Asiste:GND #PWR?
+L Asiste:GND #PWR0104
 U 1 1 5B9387C2
 P 4800 3050
-F 0 "#PWR?" H 4800 2800 50  0001 C CNN
+F 0 "#PWR0104" H 4800 2800 50  0001 C CNN
 F 1 "GND" V 4805 2922 50  0000 R CNN
 F 2 "" H 4800 3050 50  0001 C CNN
@@
 	4400 3050 4700 3050
 $Comp
-L Asiste:C_0603_1uF C?
+L Asiste:C_0603_1uF C101
 U 1 1 5B93A003
 P 4700 2850
-F 0 "C?" H 4815 2896 50  0000 L CNN
+F 0 "C101" H 4815 2896 50  0000 L CNN
 F 1 "C_0603_1uF" H 4500 2300 50  0001 L CNN
 F 2 "ASISTE:C_0603" H 4750 2600 50  0001 C CNN
@@
 	4700 3050 4800 3050
 $Comp
-L Asiste:SW_SPST SW?
+L Asiste:SW_SPST SW101
 U 1 1 5B897F2A
 P 3350 3300
-F 0 "SW?" V 3304 3398 50  0000 L CNN
+F 0 "SW101" V 3304 3398 50  0000 L CNN
 F 1 "SW_SPST" V 3395 3398 50  0000 L CNN
 F 2 "ASISTE:SW_SPST_PTS810" H 3400 3100 50  0001 C CNN
@@
 $EndComp
 $Comp
-L Asiste:R_0402_100 R?
+L Asiste:R_0402_100 R104
 U 1 1 5B89881E
 P 3350 2850
-F 0 "R?" H 3420 2896 50  0000 L CNN
+F 0 "R104" H 3420 2896 50  0000 L CNN
 F 1 "R_0402_100" H 3350 2300 50  0001 C CNN
 F 2 "ASISTE:R_0402" H 3350 2400 50  0001 C CNN
@@
 Connection ~ 4700 2600
 $Comp
-L Asiste:VCC #PWR?
+L Asiste:VCC #PWR0103
 U 1 1 5B93814B
 P 4700 2600
-F 0 "#PWR?" H 4700 2450 50  0001 C CNN
+F 0 "#PWR0103" H 4700 2450 50  0001 C CNN
 F 1 "VCC" H 4715 2773 50  0000 C CNN
 F 2 "" H 4700 2600 50  0001 C CNN
@@
 	3350 3000 3350 3050
 $Comp
-L Asiste:GND #PWR?
+L Asiste:GND #PWR0102
 U 1 1 5B89A405
 P 3350 3600
-F 0 "#PWR?" H 3350 3350 50  0001 C CNN
+F 0 "#PWR0102" H 3350 3350 50  0001 C CNN
 F 1 "GND" H 3200 3550 50  0000 C CNN
 F 2 "" H 3350 3600 50  0001 C CNN
@@
 Wire Wire Line
 	3350 3050 3350 3100
+$Sheet
+S 5250 3000 1950 1850
+U 5B56C637
+F0 "micro" 60
+F1 "micro.sch" 60
+F2 "MCU_SDA2" B R 7200 4650 60
+F3 "MCU_SCL2" O R 7200 4750 60
+F4 "MPU_PROG_RX" I L 5250 3250 60
+F5 "MCU_PROG_TX" I L 5250 3150 60
+F6 "MCU_DEBUG_SWCLK" I L 5250 3350 60
+F7 "MCU_DEBUG_SWDIO" I L 5250 3450 60
+F8 "LED_GREEN" O L 5250 3850 60
+F9 "LED_RED" O L 5250 3750 60
+F10 "LED_BLUE" O L 5250 3950 60
+F11 "PWR_EN" O L 5250 4450 60
+F12 "BAT_CHG_STAT" I L 5250 4550 60
+F13 "BUTTON" I L 5250 3650 60
+F14 "BAT_SENSE" I L 5250 4650 60
+F15 "HR_~INT" I R 7200 4550 60
+F16 "TMP_ALERT" I R 7200 4050 60
+F17 "IMU_INT" I R 7200 3150 60
+F18 "IMU_SDA" B R 7200 3250 60
+F19 "IMU_SCL" O R 7200 3350 60
+$EndSheet
 $EndSCHEMATC

Commit message: Añadido botón y otros
Changed lines of the file:
@@
 	7200 3150 8250 3150
 Wire Wire Line
-	7200 3250 7550 3250
-Wire Wire Line
-	7200 3350 7450 3350
-Wire Wire Line
 	7200 4550 8250 4550
 Wire Wire Line
-	7200 4650 8250 4650
-Wire Wire Line
-	7200 4750 8250 4750
+	7200 4650 7550 4650
+Wire Wire Line
+	7200 4750 7650 4750
 Wire Wire Line
 	4150 4650 5250 4650
@@
 	7200 4050 8250 4050
 Wire Wire Line
-	8250 3950 7450 3950
-Wire Wire Line
-	7450 3950 7450 3350
-Connection ~ 7450 3350
-Wire Wire Line
-	7450 3350 8250 3350
+	8250 3950 7650 3950
 Wire Wire Line
 	8250 3850 7550 3850
-Wire Wire Line
-	7550 3850 7550 3250
-Connection ~ 7550 3250
-Wire Wire Line
-	7550 3250 8250 3250
 $Comp
 L Asiste:LED_ARGB D101
@@
 F19 "IMU_SCL" O R 7200 3350 60
 $EndSheet
+Wire Wire Line
+	7200 3250 8250 3250
+Wire Wire Line
+	7200 3350 8250 3350
+Wire Wire Line
+	7550 3850 7550 4650
+Connection ~ 7550 4650
+Wire Wire Line
+	7550 4650 8250 4650
+Wire Wire Line
+	7650 3950 7650 4750
+Connection ~ 7650 4750
+Wire Wire Line
+	7650 4750 8250 4750
 $EndSCHEMATC

Commit message: Esquemáticos totalmente terminados y revisados PCB a falta de routear el puerto de programación
Parts:
- renumbered C101 to C1, D101 to D1, PROG101 to PROG1, R101 to R1, R102 to R2, R103 to R3, R104 to R4, SW101 to SW1
Connections:
- net labels removed: VCC
- no-connect marks 0 -> 1
Changed lines of the file:
@@
 F2 "BAT_CHG_STAT" O R 4150 4550 60
 F3 "BAT_SENSE" O R 4150 4650 60
-F4 "PWR_EN" I R 4150 4450 60
 $EndSheet
 $Sheet
@@
 	8250 3850 7550 3850
 $Comp
-L Asiste:LED_ARGB D101
+L Asiste:LED_ARGB D1
 U 1 1 5B7F5EAD
 P 2500 2850
-F 0 "D101" H 2500 2383 50  0000 C CNN
+F 0 "D1" H 2500 2383 50  0000 C CNN
 F 1 "LED_ARGB" H 2500 2474 50  0000 C CNN
 F 2 "ASISTE:LED_Cree-PLCC4_2x2mm_CW" H 2500 2250 50  0001 C CNN
@@
 	2500 2550 2500 2600
 $Comp
-L Asiste:+3V3 #PWR0101
+L Asiste:+3V3 #PWR01
 U 1 1 5B7F63F5
 P 2500 2550
-F 0 "#PWR0101" H 2500 2400 50  0001 C CNN
+F 0 "#PWR01" H 2500 2400 50  0001 C CNN
 F 1 "+3V3" H 2515 2723 50  0000 C CNN
 F 2 "" H 2500 2550 50  0001 C CNN
@@
 $EndComp
 $Comp
-L Asiste:R_0402_100 R103
+L Asiste:R_0402_100 R3
 U 1 1 5B787251
 P 2850 3300
-F 0 "R103" H 2920 3346 50  0000 L CNN
+F 0 "R3" H 2920 3346 50  0000 L CNN
 F 1 "R_0402_100" H 2850 2750 50  0001 C CNN
 F 2 "ASISTE:R_0402" H 2850 2850 50  0001 C CNN
@@
 $EndComp
 $Comp
-L Asiste:R_0402_33 R102
+L Asiste:R_0402_33 R2
 U 1 1 5B78744C
 P 2500 3300
-F 0 "R102" H 2570 3346 50  0000 L CNN
+F 0 "R2" H 2570 3346 50  0000 L CNN
 F 1 "R_0402_33" H 2500 2750 50  0001 C CNN
 F 2 "ASISTE:R_0402" H 2500 2850 50  0001 C CNN
@@
 $EndComp
 $Comp
-L Asiste:R_0402_33 R101
+L Asiste:R_0402_33 R1
 U 1 1 5B7874B2
 P 2150 3300
-F 0 "R101" H 2220 3346 50  0000 L CNN
+F 0 "R1" H 2220 3346 50  0000 L CNN
 F 1 "R_0402_33" H 2150 2750 50  0001 C CNN
 F 2 "ASISTE:R_0402" H 2150 2850 50  0001 C CNN
@@
 	2850 3050 2850 3150
 Wire Wire Line
-	5250 4450 4150 4450
-Wire Wire Line
 	5250 4550 4150 4550
 $Comp
-L Asiste:SMD_01x06 PROG101
+L Asiste:SMD_01x06 PROG1
 U 1 1 5B936A3E
 P 4200 3150
-F 0 "PROG101" H 4300 3500 50  0000 C CNN
+F 0 "PROG1" H 4300 3500 50  0000 C CNN
 F 1 "SMD_01x06" H 4200 2750 50  0001 C CNN
 F 2 "ASISTE:SMD_PROG" H 4100 3350 50  0001 C CNN
@@
 	4400 2950 4500 2950
 $Comp
-L Asiste:GND #PWR0104
+L Asiste:GND #PWR04
 U 1 1 5B9387C2
 P 4800 3050
-F 0 "#PWR0104" H 4800 2800 50  0001 C CNN
+F 0 "#PWR04" H 4800 2800 50  0001 C CNN
 F 1 "GND" V 4805 2922 50  0000 R CNN
 F 2 "" H 4800 3050 50  0001 C CNN
@@
 	4400 3050 4700 3050
 $Comp
-L Asiste:C_0603_1uF C101
+L Asiste:C_0603_1uF C1
 U 1 1 5B93A003
 P 4700 2850
-F 0 "C101" H 4815 2896 50  0000 L CNN
+F 0 "C1" H 4815 2896 50  0000 L CNN
 F 1 "C_0603_1uF" H 4500 2300 50  0001 L CNN
 F 2 "ASISTE:C_0603" H 4750 2600 50  0001 C CNN
@@
 	4500 2600 4500 2950
 Wire Wire Line
-	4700 2700 4700 2600
-Wire Wire Line
 	4500 2600 4700 2600
 Wire Wire Line
@@
 	4700 3050 4800 3050
 $Comp
-L Asiste:SW_SPST SW101
+L Asiste:SW_SPST SW1
 U 1 1 5B897F2A
 P 3350 3300
-F 0 "SW101" V 3304 3398 50  0000 L CNN
+F 0 "SW1" V 3304 3398 50  0000 L CNN
 F 1 "SW_SPST" V 3395 3398 50  0000 L CNN
 F 2 "ASISTE:SW_SPST_PTS810" H 3400 3100 50  0001 C CNN
@@
 $EndComp
 $Comp
-L Asiste:R_0402_100 R104
+L Asiste:R_0402_100 R4
 U 1 1 5B89881E
 P 3350 2850
-F 0 "R104" H 3420 2896 50  0000 L CNN
+F 0 "R4" H 3420 2896 50  0000 L CNN
 F 1 "R_0402_100" H 3350 2300 50  0001 C CNN
 F 2 "ASISTE:R_0402" H 3350 2400 50  0001 C CNN
@@
 Wire Wire Line
 	2500 2600 2500 2650
-Connection ~ 4700 2600
-$Comp
-L Asiste:VCC #PWR0103
-U 1 1 5B93814B
-P 4700 2600
-F 0 "#PWR0103" H 4700 2450 50  0001 C CNN
-F 1 "VCC" H 4715 2773 50  0000 C CNN
-F 2 "" H 4700 2600 50  0001 C CNN
-F 3 "" H 4700 2600 50  0001 C CNN
-	1    4700 2600
-	1    0    0    -1
-$EndComp
 Wire Wire Line
 	3350 3000 3350 3050
 $Comp
-L Asiste:GND #PWR0102
+L Asiste:GND #PWR02
 U 1 1 5B89A405
 P 3350 3600
-F 0 "#PWR0102" H 3350 3350 50  0001 C CNN
+F 0 "#PWR02" H 3350 3350 50  0001 C CNN
 F 1 "GND" H 3200 3550 50  0000 C CNN
 F 2 "" H 3350 3600 50  0001 C CNN
@@
 F9 "LED_RED" O L 5250 3750 60
 F10 "LED_BLUE" O L 5250 3950 60
-F11 "PWR_EN" O L 5250 4450 60
-F12 "BAT_CHG_STAT" I L 5250 4550 60
-F13 "BUTTON" I L 5250 3650 60
-F14 "BAT_SENSE" I L 5250 4650 60
-F15 "HR_~INT" I R 7200 4550 60
-F16 "TMP_ALERT" I R 7200 4050 60
-F17 "IMU_INT" I R 7200 3150 60
-F18 "IMU_SDA" B R 7200 3250 60
-F19 "IMU_SCL" O R 7200 3350 60
+F11 "BAT_CHG_STAT" I L 5250 4550 60
+F12 "BUTTON" I L 5250 3650 60
+F13 "BAT_SENSE" I L 5250 4650 60
+F14 "HR_~INT" I R 7200 4550 60
+F15 "TMP_ALERT" I R 7200 4050 60
+F16 "IMU_INT" I R 7200 3150 60
+F17 "IMU_SDA" B R 7200 3250 60
+F18 "IMU_SCL" O R 7200 3350 60
 $EndSheet
 Wire Wire Line
@@
 Wire Wire Line
 	7650 4750 8250 4750
+$Comp
+L Asiste:+3V3 #PWR03
+U 1 1 5B980752
+P 4700 2550
+F 0 "#PWR03" H 4700 2400 50  0001 C CNN
+F 1 "+3V3" H 4750 2750 50  0000 C CNN
+F 2 "" H 4700 2550 50  0001 C CNN
+F 3 "" H 4700 2550 50  0001 C CNN
+	1    4700 2550
+	1    0    0    -1
+$EndComp
+Connection ~ 4700 2600
+Wire Wire Line
+	4700 2600 4700 2700
+Wire Wire Line
+	4700 2550 4700 2600
+NoConn ~ 6150 4200
 $EndSCHEMATC

Commit message: Actualizando
Parts:
- removed C1: C_0603_1uF, ASISTE:C_0603, symbol Asiste:C_0603_1uF
Connections:
- wire segments 48 -> 42
Changed lines of the file:
@@
 U 5B55F5BB
 F0 "heartRate" 60
-F1 "heartRatesch.sch" 60
+F1 "heartRate.sch" 60
 F2 "HR_~INT" O L 8250 4550 60
 F3 "HR_SCL" I L 8250 4750 60
@@
 	4400 3450 5250 3450
 Wire Wire Line
-	4400 2950 4500 2950
+	4400 2950 4800 2950
 $Comp
 L Asiste:GND #PWR04
@@
 P 4800 3050
 F 0 "#PWR04" H 4800 2800 50  0001 C CNN
-F 1 "GND" V 4805 2922 50  0000 R CNN
+F 1 "GND" V 4800 2900 50  0000 R CNN
 F 2 "" H 4800 3050 50  0001 C CNN
 F 3 "" H 4800 3050 50  0001 C CNN
@@
 	0    -1   -1   0
 $EndComp
-Wire Wire Line
-	4400 3050 4700 3050
-$Comp
-L Asiste:C_0603_1uF C1
-U 1 1 5B93A003
-P 4700 2850
-F 0 "C1" H 4815 2896 50  0000 L CNN
-F 1 "C_0603_1uF" H 4500 2300 50  0001 L CNN
-F 2 "ASISTE:C_0603" H 4750 2600 50  0001 C CNN
-F 3 "https://www.mouser.es/datasheet/2/396/mlcc02_e-1307760.pdf" H 5250 2500 50  0001 C CNN
-F 4 "LMK107B7105KAHT" H 4700 2400 60  0001 C CNN "man#"
-F 5 "1uF" H 4815 2805 50  0000 L CNN "Capacitance"
-F 6 "10V" H 4700 2400 60  0001 C CNN "Voltage"
-	1    4700 2850
-	1    0    0    -1
-$EndComp
-Wire Wire Line
-	4500 2600 4500 2950
-Wire Wire Line
-	4500 2600 4700 2600
-Wire Wire Line
-	4700 3000 4700 3050
-Connection ~ 4700 3050
-Wire Wire Line
-	4700 3050 4800 3050
 $Comp
 L Asiste:SW_SPST SW1
@@
 F2 "MCU_SDA2" B R 7200 4650 60
 F3 "MCU_SCL2" O R 7200 4750 60
-F4 "MPU_PROG_RX" I L 5250 3250 60
-F5 "MCU_PROG_TX" I L 5250 3150 60
-F6 "MCU_DEBUG_SWCLK" I L 5250 3350 60
-F7 "MCU_DEBUG_SWDIO" I L 5250 3450 60
-F8 "LED_GREEN" O L 5250 3850 60
-F9 "LED_RED" O L 5250 3750 60
-F10 "LED_BLUE" O L 5250 3950 60
-F11 "BAT_CHG_STAT" I L 5250 4550 60
-F12 "BUTTON" I L 5250 3650 60
-F13 "BAT_SENSE" I L 5250 4650 60
-F14 "HR_~INT" I R 7200 4550 60
-F15 "TMP_ALERT" I R 7200 4050 60
-F16 "IMU_INT" I R 7200 3150 60
-F17 "IMU_SDA" B R 7200 3250 60
-F18 "IMU_SCL" O R 7200 3350 60
+F4 "MCU_PROG_TX" I L 5250 3150 60
+F5 "MCU_DEBUG_SWCLK" I L 5250 3350 60
+F6 "MCU_DEBUG_SWDIO" I L 5250 3450 60
+F7 "LED_GREEN" O L 5250 3850 60
+F8 "LED_RED" O L 5250 3750 60
+F9 "LED_BLUE" O L 5250 3950 60
+F10 "BAT_CHG_STAT" I L 5250 4550 60
+F11 "BUTTON" I L 5250 3650 60
+F12 "BAT_SENSE" I L 5250 4650 60
+F13 "HR_~INT" I R 7200 4550 60
+F14 "TMP_ALERT" I R 7200 4050 60
+F15 "IMU_INT" I R 7200 3150 60
+F16 "IMU_SDA" B R 7200 3250 60
+F17 "IMU_SCL" O R 7200 3350 60
+F18 "MCU_PROG_RX" I L 5250 3250 60
 $EndSheet
 Wire Wire Line
@@
 L Asiste:+3V3 #PWR03
 U 1 1 5B980752
-P 4700 2550
-F 0 "#PWR03" H 4700 2400 50  0001 C CNN
-F 1 "+3V3" H 4750 2750 50  0000 C CNN
-F 2 "" H 4700 2550 50  0001 C CNN
-F 3 "" H 4700 2550 50  0001 C CNN
-	1    4700 2550
-	1    0    0    -1
-$EndComp
-Connection ~ 4700 2600
-Wire Wire Line
-	4700 2600 4700 2700
-Wire Wire Line
-	4700 2550 4700 2600
+P 4800 2950
+F 0 "#PWR03" H 4800 2800 50  0001 C CNN
+F 1 "+3V3" V 4800 3150 50  0000 C CNN
+F 2 "" H 4800 2950 50  0001 C CNN
+F 3 "" H 4800 2950 50  0001 C CNN
+	1    4800 2950
+	0    1    1    0
+$EndComp
 NoConn ~ 6150 4200
+Wire Wire Line
+	4400 3050 4800 3050
 $EndSCHEMATC
