File: heartRatesch.sch (KiCad schematic (older format))
At the start: 9 parts

Commit message: Terminado esquemático. Falta revisar
Connections:
- net labels added: +3V3
- net labels removed: +5V
Changed lines of the file:
@@
 	4950 3400 4950 3250
 Connection ~ 4950 3250
-$Comp
-L Asiste:+5V #PWR?
-U 1 1 5B7961FD
-P 6450 2350
-F 0 "#PWR?" H 6450 2200 50  0001 C CNN
-F 1 "+5V" H 6465 2523 50  0000 C CNN
-F 2 "" H 6450 2350 50  0001 C CNN
-F 3 "" H 6450 2350 50  0001 C CNN
-	1    6450 2350
-	1    0    0    -1
-$EndComp
 Wire Wire Line
 	6050 2900 6450 2900
-Wire Wire Line
-	6450 2900 6450 2350
 $Comp
 L Asiste:MAX30105 IC?
@@
 Wire Wire Line
 	5950 4050 5950 4100
+Wire Wire Line
+	6450 2900 6450 2350
+$Comp
+L Asiste:+3V3 #PWR?
+U 1 1 5B8B05EF
+P 6450 2350
+F 0 "#PWR?" H 6450 2200 50  0001 C CNN
+F 1 "+3V3" H 6465 2523 50  0000 C CNN
+F 2 "" H 6450 2350 50  0001 C CNN
+F 3 "" H 6450 2350 50  0001 C CNN
+	1    6450 2350
+	1    0    0    -1
+$EndComp
 $EndSCHEMATC

Commit message: Esquemático parcialmente revisado. Falta revisar pines y correspondencia con footprints
Parts:
- removed IC?: MAX30105, OptoDevice:Maxim_OLGA-14_3.3x5.6mm_P0.8mm, symbol Asiste:MAX30105
- added IC201: MAX30105, ASISTE:Maxim_OLGA-14_3.3x5.6mm_P0.8mm, symbol Asiste:MAX30105
- gave numbers to parts that had none: 8
Connections:
- wire segments 42 -> 44
- no-connect marks 0 -> 3
Changed lines of the file:
@@
 $EndDescr
 $Comp
-L Asiste:C_0603_4.7uF C?
+L Asiste:C_0603_4.7uF C201
 U 1 1 5B5650BB
 P 5750 2650
-F 0 "C?" H 5636 2604 50  0000 R CNN
+F 0 "C201" H 5636 2604 50  0000 R CNN
 F 1 "C_0603_4.7uF" H 5550 2100 50  0001 L CNN
 F 2 "ASISTE:C_0603" H 5800 2400 50  0001 C CNN
@@
 $EndComp
 Wire Wire Line
-	5750 2800 5750 3000
-$Comp
-L Asiste:C_0603_10uF C?
+	5750 2800 5750 2850
+$Comp
+L Asiste:C_0603_10uF C202
 U 1 1 5B565E1E
 P 6050 2650
-F 0 "C?" H 6165 2696 50  0000 L CNN
+F 0 "C202" H 6165 2696 50  0000 L CNN
 F 1 "C_0603_10uF" H 5850 2100 50  0001 L CNN
 F 2 "ASISTE:C_0603" H 6100 2400 50  0001 C CNN
@@
 	6050 2900 6050 3000
 $Comp
-L Asiste:GND #PWR?
+L Asiste:GND #PWR0203
 U 1 1 5B565EEE
 P 5300 2500
-F 0 "#PWR?" H 5300 2250 50  0001 C CNN
+F 0 "#PWR0203" H 5300 2250 50  0001 C CNN
 F 1 "GND" H 5305 2327 50  0000 C CNN
 F 2 "" H 5300 2500 50  0001 C CNN
@@
 	5750 2350 6050 2350
 $Comp
-L Asiste:R_0402_10k R?
+L Asiste:R_0402_10k R201
 U 1 1 5B566757
 P 4950 3000
-F 0 "R?" H 5020 3046 50  0000 L CNN
+F 0 "R201" H 5020 3046 50  0000 L CNN
 F 1 "R_0402_10k" H 4950 2450 50  0001 C CNN
 F 2 "ASISTE:R_0402" H 4950 2550 50  0001 C CNN
@@
 	4950 3250 4950 3150
 $Comp
-L Asiste:R_0402_10k R?
+L Asiste:R_0402_10k R202
 U 1 1 5B56687F
 P 4950 4050
-F 0 "R?" H 5020 4096 50  0000 L CNN
+F 0 "R202" H 5020 4096 50  0000 L CNN
 F 1 "R_0402_10k" H 4950 3500 50  0001 C CNN
 F 2 "ASISTE:R_0402" H 4950 3600 50  0001 C CNN
@@
 $EndComp
 $Comp
-L Asiste:R_0402_10k R?
+L Asiste:R_0402_10k R203
 U 1 1 5B566B71
 P 6850 3200
-F 0 "R?" H 6920 3246 50  0000 L CNN
+F 0 "R203" H 6920 3246 50  0000 L CNN
 F 1 "R_0402_10k" H 6850 2650 50  0001 C CNN
 F 2 "ASISTE:R_0402" H 6850 2750 50  0001 C CNN
@@
 	6850 2950 6850 3000
 $Comp
-L Asiste:GND #PWR?
+L Asiste:GND #PWR0205
 U 1 1 5B5673C7
 P 5950 4100
-F 0 "#PWR?" H 5950 3850 50  0001 C CNN
+F 0 "#PWR0205" H 5950 3850 50  0001 C CNN
 F 1 "GND" H 5955 3927 50  0000 C CNN
 F 2 "" H 5950 4100 50  0001 C CNN
@@
 HR_SDA
 $Comp
-L Asiste:BSS138 Q?
+L Asiste:BSS138 Q201
 U 1 1 5B747A70
 P 4000 3150
-F 0 "Q?" V 3900 2950 50  0000 C CNN
+F 0 "Q201" V 3900 2950 50  0000 C CNN
 F 1 "BSS138" V 4000 2850 50  0000 C CNN
 F 2 "ASISTE:SOT-23" H 4200 3075 50  0001 L CIN
@@
 $EndComp
 $Comp
-L Asiste:BSS138 Q?
+L Asiste:BSS138 Q202
 U 1 1 5B749C53
 P 4000 3800
-F 0 "Q?" V 3950 3600 50  0000 C CNN
+F 0 "Q202" V 3950 3600 50  0000 C CNN
 F 1 "BSS138" V 3850 3500 50  0000 C CNN
 F 2 "ASISTE:SOT-23" H 4200 3725 50  0001 L CIN
@@
 	3450 3250 3800 3250
 $Comp
-L Asiste:BSS138 Q?
+L Asiste:BSS138 Q203
 U 1 1 5B750668
 P 7650 3300
-F 0 "Q?" V 7900 3300 50  0000 C CNN
+F 0 "Q203" V 7900 3300 50  0000 C CNN
 F 1 "BSS138" V 7991 3300 50  0000 C CNN
 F 2 "ASISTE:SOT-23" H 7850 3225 50  0001 L CIN
@@
 	6850 3000 6850 3050
 $Comp
-L Asiste:+1V8 #PWR?
+L Asiste:+1V8 #PWR0201
 U 1 1 5B753557
 P 4000 2600
-F 0 "#PWR?" H 4000 2450 50  0001 C CNN
+F 0 "#PWR0201" H 4000 2450 50  0001 C CNN
 F 1 "+1V8" H 4015 2773 50  0000 C CNN
 F 2 "" H 4000 2600 50  0001 C CNN
@@
 $EndComp
 $Comp
-L Asiste:+1V8 #PWR?
+L Asiste:+1V8 #PWR0207
 U 1 1 5B753634
 P 6850 2950
-F 0 "#PWR?" H 6850 2800 50  0001 C CNN
+F 0 "#PWR0207" H 6850 2800 50  0001 C CNN
 F 1 "+1V8" H 6865 3123 50  0000 C CNN
 F 2 "" H 6850 2950 50  0001 C CNN
@@
 	4000 4000 4000 4300
 $Comp
-L Asiste:+1V8 #PWR?
+L Asiste:+1V8 #PWR0202
 U 1 1 5B78ABA9
 P 4000 4450
-F 0 "#PWR?" H 4000 4300 50  0001 C CNN
+F 0 "#PWR0202" H 4000 4300 50  0001 C CNN
 F 1 "+1V8" H 4015 4623 50  0000 C CNN
 F 2 "" H 4000 4450 50  0001 C CNN
@@
 Wire Wire Line
 	6050 2900 6450 2900
-$Comp
-L Asiste:MAX30105 IC?
-U 1 1 5B77F5B0
-P 6050 3500
-F 0 "IC?" H 5600 3950 50  0000 R CNN
-F 1 "MAX30105" H 5850 3050 50  0000 R CNN
-F 2 "OptoDevice:Maxim_OLGA-14_3.3x5.6mm_P0.8mm" H 6050 2650 50  0001 C CNN
-F 3 "https://datasheets.maximintegrated.com/en/ds/MAX30105.pdf" H 6150 2550 50  0001 C CNN
-F 4 "MAX30105EFD+" H 6050 2450 60  0001 C CNN "man#"
-	1    6050 3500
-	1    0    0    -1
-$EndComp
 Wire Wire Line
 	5950 4000 5950 4050
@@
 	6450 2900 6450 2350
 $Comp
-L Asiste:+3V3 #PWR?
+L Asiste:+3V3 #PWR0206
 U 1 1 5B8B05EF
 P 6450 2350
-F 0 "#PWR?" H 6450 2200 50  0001 C CNN
+F 0 "#PWR0206" H 6450 2200 50  0001 C CNN
 F 1 "+3V3" H 6465 2523 50  0000 C CNN
 F 2 "" H 6450 2350 50  0001 C CNN
@@
 	1    0    0    -1
 $EndComp
+NoConn ~ 6650 3600
+NoConn ~ 6650 3700
+NoConn ~ 6650 3800
+$Comp
+L Asiste:+1V8 #PWR0204
+U 1 1 5B8A2221
+P 5600 2850
+F 0 "#PWR0204" H 5600 2700 50  0001 C CNN
+F 1 "+1V8" V 5615 2978 50  0000 L CNN
+F 2 "" H 5600 2850 50  0001 C CNN
+F 3 "" H 5600 2850 50  0001 C CNN
+	1    5600 2850
+	0    -1   -1   0
+$EndComp
+Wire Wire Line
+	5600 2850 5750 2850
+Connection ~ 5750 2850
+Wire Wire Line
+	5750 2850 5750 3000
+$Comp
+L Asiste:MAX30105 IC201
+U 1 1 5B8C1E27
+P 6050 3500
+F 0 "IC201" H 5450 3950 50  0000 R CNN
+F 1 "MAX30105" H 6500 3950 50  0000 R CNN
+F 2 "ASISTE:Maxim_OLGA-14_3.3x5.6mm_P0.8mm" H 6050 2650 50  0001 C CNN
+F 3 "https://datasheets.maximintegrated.com/en/ds/MAX30105.pdf" H 6150 2550 50  0001 C CNN
+F 4 "MAX30105EFD+" H 6050 2450 60  0001 C CNN "man#"
+	1    6050 3500
+	1    0    0    -1
+$EndComp

Commit message: Esquemáticos totalmente terminados y revisados PCB a falta de routear el puerto de programación
Parts:
- removed C202: C_0603_10uF, ASISTE:C_0603, symbol Asiste:C_0603_10uF
- removed Q201, Q202, Q203: BSS138, ASISTE:SOT-23, symbol Asiste:BSS138
- added C3: C_0603_10uF, ASISTE:C_0603, symbol Asiste:C_0603_10uF
- added Q1, Q2, Q3: NTK3134NT1G, ASISTE:SOT-723, symbol Asiste:NTK3134NT1G
- renumbered C201 to C2, IC201 to IC1, R201 to R5, R202 to R6, R203 to R7
Changed lines of the file:
@@
 $EndDescr
 $Comp
-L Asiste:C_0603_4.7uF C201
+L Asiste:C_0603_4.7uF C2
 U 1 1 5B5650BB
 P 5750 2650
-F 0 "C201" H 5636 2604 50  0000 R CNN
+F 0 "C2" H 5636 2604 50  0000 R CNN
 F 1 "C_0603_4.7uF" H 5550 2100 50  0001 L CNN
 F 2 "ASISTE:C_0603" H 5800 2400 50  0001 C CNN
@@
 Wire Wire Line
 	5750 2800 5750 2850
-$Comp
-L Asiste:C_0603_10uF C202
-U 1 1 5B565E1E
-P 6050 2650
-F 0 "C202" H 6165 2696 50  0000 L CNN
-F 1 "C_0603_10uF" H 5850 2100 50  0001 L CNN
-F 2 "ASISTE:C_0603" H 6100 2400 50  0001 C CNN
-F 3 "https://eu.mouser.com/datasheet/2/281/murata_03052018_GRM_Series_1-1310166.pdf" H 6600 2300 50  0001 C CNN
-F 4 "GRM188R60J106KE47D" H 6050 2000 60  0001 C CNN "man#"
-F 5 "10uF" H 6165 2605 50  0000 L CNN "Capacitance"
-F 6 "6V3" H 6050 2200 60  0001 C CNN "Voltage"
-	1    6050 2650
-	1    0    0    -1
-$EndComp
 Wire Wire Line
 	6050 2800 6050 2900
@@
 	6050 2900 6050 3000
 $Comp
-L Asiste:GND #PWR0203
+L Asiste:GND #PWR07
 U 1 1 5B565EEE
 P 5300 2500
-F 0 "#PWR0203" H 5300 2250 50  0001 C CNN
+F 0 "#PWR07" H 5300 2250 50  0001 C CNN
 F 1 "GND" H 5305 2327 50  0000 C CNN
 F 2 "" H 5300 2500 50  0001 C CNN
@@
 	5750 2350 6050 2350
 $Comp
-L Asiste:R_0402_10k R201
+L Asiste:R_0402_10k R5
 U 1 1 5B566757
 P 4950 3000
-F 0 "R201" H 5020 3046 50  0000 L CNN
+F 0 "R5" H 5020 3046 50  0000 L CNN
 F 1 "R_0402_10k" H 4950 2450 50  0001 C CNN
 F 2 "ASISTE:R_0402" H 4950 2550 50  0001 C CNN
@@
 	4950 3250 4950 3150
 $Comp
-L Asiste:R_0402_10k R202
+L Asiste:R_0402_10k R6
 U 1 1 5B56687F
 P 4950 4050
-F 0 "R202" H 5020 4096 50  0000 L CNN
+F 0 "R6" H 5020 4096 50  0000 L CNN
 F 1 "R_0402_10k" H 4950 3500 50  0001 C CNN
 F 2 "ASISTE:R_0402" H 4950 3600 50  0001 C CNN
@@
 $EndComp
 $Comp
-L Asiste:R_0402_10k R203
+L Asiste:R_0402_10k R7
 U 1 1 5B566B71
 P 6850 3200
-F 0 "R203" H 6920 3246 50  0000 L CNN
+F 0 "R7" H 6920 3246 50  0000 L CNN
 F 1 "R_0402_10k" H 6850 2650 50  0001 C CNN
 F 2 "ASISTE:R_0402" H 6850 2750 50  0001 C CNN
@@
 	6850 2950 6850 3000
 $Comp
-L Asiste:GND #PWR0205
+L Asiste:GND #PWR09
 U 1 1 5B5673C7
 P 5950 4100
-F 0 "#PWR0205" H 5950 3850 50  0001 C CNN
+F 0 "#PWR09" H 5950 3850 50  0001 C CNN
 F 1 "GND" H 5955 3927 50  0000 C CNN
 F 2 "" H 5950 4100 50  0001 C CNN
@@
 Text HLabel 3450 3700 0    60   BiDi ~ 0
 HR_SDA
-$Comp
-L Asiste:BSS138 Q201
-U 1 1 5B747A70
-P 4000 3150
-F 0 "Q201" V 3900 2950 50  0000 C CNN
-F 1 "BSS138" V 4000 2850 50  0000 C CNN
-F 2 "ASISTE:SOT-23" H 4200 3075 50  0001 L CIN
-F 3 "https://www.fairchildsemi.com/datasheets/BS/BSS138.pdf" H 4200 3225 50  0001 L CNN
-F 4 "BSS138" H 4200 3000 60  0001 L CNN "man#"
-	1    4000 3150
-	0    -1   1    0
-$EndComp
-$Comp
-L Asiste:BSS138 Q202
-U 1 1 5B749C53
-P 4000 3800
-F 0 "Q202" V 3950 3600 50  0000 C CNN
-F 1 "BSS138" V 3850 3500 50  0000 C CNN
-F 2 "ASISTE:SOT-23" H 4200 3725 50  0001 L CIN
-F 3 "https://www.fairchildsemi.com/datasheets/BS/BSS138.pdf" H 4200 3875 50  0001 L CNN
-F 4 "BSS138" H 4200 3650 60  0001 L CNN "man#"
-	1    4000 3800
-	0    -1   -1   0
-$EndComp
 Wire Wire Line
 	4200 3250 4950 3250
@@
 Wire Wire Line
 	3450 3250 3800 3250
-$Comp
-L Asiste:BSS138 Q203
-U 1 1 5B750668
-P 7650 3300
-F 0 "Q203" V 7900 3300 50  0000 C CNN
-F 1 "BSS138" V 7991 3300 50  0000 C CNN
-F 2 "ASISTE:SOT-23" H 7850 3225 50  0001 L CIN
-F 3 "https://www.fairchildsemi.com/datasheets/BS/BSS138.pdf" H 7850 3375 50  0001 L CNN
-F 4 "BSS138" H 7850 3150 60  0001 L CNN "man#"
-	1    7650 3300
-	0    1    1    0
-$EndComp
 Wire Wire Line
 	6850 3400 7450 3400
@@
 	6850 3000 6850 3050
 $Comp
-L Asiste:+1V8 #PWR0201
+L Asiste:+1V8 #PWR05
 U 1 1 5B753557
 P 4000 2600
-F 0 "#PWR0201" H 4000 2450 50  0001 C CNN
+F 0 "#PWR05" H 4000 2450 50  0001 C CNN
 F 1 "+1V8" H 4015 2773 50  0000 C CNN
 F 2 "" H 4000 2600 50  0001 C CNN
@@
 $EndComp
 $Comp
-L Asiste:+1V8 #PWR0207
+L Asiste:+1V8 #PWR011
 U 1 1 5B753634
 P 6850 2950
-F 0 "#PWR0207" H 6850 2800 50  0001 C CNN
+F 0 "#PWR011" H 6850 2800 50  0001 C CNN
 F 1 "+1V8" H 6865 3123 50  0000 C CNN
 F 2 "" H 6850 2950 50  0001 C CNN
@@
 	4000 4000 4000 4300
 $Comp
-L Asiste:+1V8 #PWR0202
+L Asiste:+1V8 #PWR06
 U 1 1 5B78ABA9
 P 4000 4450
-F 0 "#PWR0202" H 4000 4300 50  0001 C CNN
+F 0 "#PWR06" H 4000 4300 50  0001 C CNN
 F 1 "+1V8" H 4015 4623 50  0000 C CNN
 F 2 "" H 4000 4450 50  0001 C CNN
@@
 	6450 2900 6450 2350
 $Comp
-L Asiste:+3V3 #PWR0206
+L Asiste:+3V3 #PWR010
 U 1 1 5B8B05EF
 P 6450 2350
-F 0 "#PWR0206" H 6450 2200 50  0001 C CNN
+F 0 "#PWR010" H 6450 2200 50  0001 C CNN
 F 1 "+3V3" H 6465 2523 50  0000 C CNN
 F 2 "" H 6450 2350 50  0001 C CNN
@@
 NoConn ~ 6650 3800
 $Comp
-L Asiste:+1V8 #PWR0204
+L Asiste:+1V8 #PWR08
 U 1 1 5B8A2221
 P 5600 2850
-F 0 "#PWR0204" H 5600 2700 50  0001 C CNN
+F 0 "#PWR08" H 5600 2700 50  0001 C CNN
 F 1 "+1V8" V 5615 2978 50  0000 L CNN
 F 2 "" H 5600 2850 50  0001 C CNN
@@
 	5750 2850 5750 3000
 $Comp
-L Asiste:MAX30105 IC201
+L Asiste:MAX30105 IC1
 U 1 1 5B8C1E27
 P 6050 3500
-F 0 "IC201" H 5450 3950 50  0000 R CNN
+F 0 "IC1" H 5450 3950 50  0000 R CNN
 F 1 "MAX30105" H 6500 3950 50  0000 R CNN
 F 2 "ASISTE:Maxim_OLGA-14_3.3x5.6mm_P0.8mm" H 6050 2650 50  0001 C CNN
@@
 	1    0    0    -1
 $EndComp
+$Comp
+L Asiste:NTK3134NT1G Q1
+U 1 1 5B953757
+P 4000 3150
+F 0 "Q1" V 4050 3400 50  0000 C CNN
+F 1 "NTK3134NT1G" V 4050 2750 50  0000 C CNN
+F 2 "ASISTE:SOT-723" H 4200 3075 50  0001 L CIN
+F 3 "https://www.onsemi.com/pub/Collateral/NTK3134N-D.PDF" H 4200 3225 50  0001 L CNN
+F 4 "NTK3134NT1G" H 4200 3000 60  0001 L CNN "man#"
+	1    4000 3150
+	0    -1   1    0
+$EndComp
+$Comp
+L Asiste:NTK3134NT1G Q2
+U 1 1 5B955A9D
+P 4000 3800
+F 0 "Q2" V 4050 4050 50  0000 C CNN
+F 1 "NTK3134NT1G" V 4050 3350 50  0000 C CNN
+F 2 "ASISTE:SOT-723" H 4200 3725 50  0001 L CIN
+F 3 "https://www.onsemi.com/pub/Collateral/NTK3134N-D.PDF" H 4200 3875 50  0001 L CNN
+F 4 "NTK3134NT1G" H 4200 3650 60  0001 L CNN "man#"
+	1    4000 3800
+	0    -1   -1   0
+$EndComp
+$Comp
+L Asiste:NTK3134NT1G Q3
+U 1 1 5B9575EC
+P 7650 3300
+F 0 "Q3" V 7700 3100 50  0000 C CNN
+F 1 "NTK3134NT1G" V 7700 3700 50  0000 C CNN
+F 2 "ASISTE:SOT-723" H 7850 3225 50  0001 L CIN
+F 3 "https://www.onsemi.com/pub/Collateral/NTK3134N-D.PDF" H 7850 3375 50  0001 L CNN
+F 4 "NTK3134NT1G" H 7850 3150 60  0001 L CNN "man#"
+	1    7650 3300
+	0    1    1    0
+$EndComp
+$Comp
+L Asiste:C_0603_10uF C3
+U 1 1 5B94F806
+P 6050 2650
+F 0 "C3" H 6150 2700 50  0000 L CNN
+F 1 "C_0603_10uF" H 5850 2000 50  0001 L CNN
+F 2 "ASISTE:C_0603" H 6100 2400 50  0001 C CNN
+F 3 "https://eu.mouser.com/datasheet/2/281/murata_03052018_GRM_Series_1-1310166.pdf" H 6600 2300 50  0001 C CNN
+F 4 "GRM188R60J106KE47D" H 6050 2100 60  0001 C CNN "man#"
+F 5 "10uF" H 6150 2600 50  0000 L CNN "Capacitance"
+F 6 "6.3V" H 6050 2200 60  0001 C CNN "Voltage"
+	1    6050 2650
+	1    0    0    -1
+$EndComp

Commit message: Actualizando
Parts:
- renumbered C2 to C1, C3 to C2
Changed lines of the file:
@@
 $EndDescr
 $Comp
-L Asiste:C_0603_4.7uF C2
+L Asiste:C_0603_4.7uF C1
 U 1 1 5B5650BB
 P 5750 2650
-F 0 "C2" H 5636 2604 50  0000 R CNN
+F 0 "C1" H 5636 2604 50  0000 R CNN
 F 1 "C_0603_4.7uF" H 5550 2100 50  0001 L CNN
 F 2 "ASISTE:C_0603" H 5800 2400 50  0001 C CNN
@@
 $EndComp
 $Comp
-L Asiste:C_0603_10uF C3
+L Asiste:C_0603_10uF C2
 U 1 1 5B94F806
 P 6050 2650
-F 0 "C3" H 6150 2700 50  0000 L CNN
+F 0 "C2" H 6150 2700 50  0000 L CNN
 F 1 "C_0603_10uF" H 5850 2000 50  0001 L CNN
 F 2 "ASISTE:C_0603" H 6100 2400 50  0001 C CNN
