File: imu.sch (KiCad schematic (older format))
At the start: 7 parts

Commit message: Esquemático parcialmente revisado. Falta revisar pines y correspondencia con footprints
Parts:
- gave numbers to parts that had none: 7
Changed lines of the file:
@@
 $EndDescr
 $Comp
-L Asiste:GND #PWR?
+L Asiste:GND #PWR0404
 U 1 1 5B266BE2
 P 5850 4700
-F 0 "#PWR?" H 5850 4450 50  0001 C CNN
+F 0 "#PWR0404" H 5850 4450 50  0001 C CNN
 F 1 "GND" H 5850 4550 50  0000 C CNN
 F 2 "" H 5850 4700 50  0001 C CNN
@@
 AR Path="/5B266C17" Ref="#PWR?"  Part="1"
 AR Path="/5B26151D/5B266C17" Ref="#PWR?"  Part="1"
-AR Path="/5B56C4B2/5B266C17" Ref="#PWR?"  Part="1"
-F 0 "#PWR?" H 5850 2500 50  0001 C CNN
+AR Path="/5B56C4B2/5B266C17" Ref="#PWR0403"  Part="1"
+F 0 "#PWR0403" H 5850 2500 50  0001 C CNN
 F 1 "+3V3" H 5850 2790 50  0000 C CNN
 F 2 "" H 5850 2650 50  0001 C CNN
@@
 $EndComp
 $Comp
-L Asiste:GND #PWR?
+L Asiste:GND #PWR0405
 U 1 1 5B267277
 P 7000 3100
-F 0 "#PWR?" H 7000 2850 50  0001 C CNN
+F 0 "#PWR0405" H 7000 2850 50  0001 C CNN
 F 1 "GND" H 7000 2950 50  0000 C CNN
 F 2 "" H 7000 3100 50  0001 C CNN
@@
 	4600 2950 4600 3100
 $Comp
-L Asiste:GND #PWR?
+L Asiste:GND #PWR0401
 U 1 1 5B267478
 P 4600 3100
-F 0 "#PWR?" H 4600 2850 50  0001 C CNN
+F 0 "#PWR0401" H 4600 2850 50  0001 C CNN
 F 1 "GND" H 4600 2950 50  0000 C CNN
 F 2 "" H 4600 3100 50  0001 C CNN
@@
 	6950 4150 6550 4150
 $Comp
-L Asiste:GND #PWR?
+L Asiste:GND #PWR0406
 U 1 1 5B26785D
 P 7300 4700
-F 0 "#PWR?" H 7300 4450 50  0001 C CNN
+F 0 "#PWR0406" H 7300 4450 50  0001 C CNN
 F 1 "GND" H 7300 4550 50  0000 C CNN
 F 2 "" H 7300 4700 50  0001 C CNN
@@
 Connection ~ 7300 4650
 $Comp
-L Asiste:GND #PWR?
+L Asiste:GND #PWR0402
 U 1 1 5B2678F3
 P 4950 4200
-F 0 "#PWR?" H 4950 3950 50  0001 C CNN
+F 0 "#PWR0402" H 4950 3950 50  0001 C CNN
 F 1 "GND" H 4950 4050 50  0000 C CNN
 F 2 "" H 4950 4200 50  0001 C CNN
@@
 Connection ~ 4250 3650
 $Comp
-L Asiste:C_0402_2.2nF C?
+L Asiste:C_0402_2.2nF C404
 U 1 1 5B370B27
 P 7300 4400
-F 0 "C?" H 7325 4500 50  0000 L CNN
+F 0 "C404" H 7325 4500 50  0000 L CNN
 F 1 "C_0402_2.2nF" H 7150 3850 50  0001 L CNN
 F 2 "ASISTE:C_0402" H 7350 4150 50  0001 C CNN
@@
 $EndComp
 $Comp
-L Asiste:C_0402_100nF C?
+L Asiste:C_0402_100nF C403
 U 1 1 5B370BA6
 P 6950 4400
-F 0 "C?" H 6975 4500 50  0000 L CNN
+F 0 "C403" H 6975 4500 50  0000 L CNN
 F 1 "C_0402_100nF" H 6700 3850 50  0001 L CNN
 F 2 "ASISTE:C_0402" H 7000 4150 50  0001 C CNN
@@
 $EndComp
 $Comp
-L Asiste:R_0402_10k R?
+L Asiste:R_0402_10k R401
 U 1 1 5B370C5C
 P 3950 3250
-F 0 "R?" H 3850 3400 50  0000 L CNN
+F 0 "R401" H 3850 3400 50  0000 L CNN
 F 1 "R_0402_10k" H 3950 2700 50  0001 C CNN
 F 2 "ASISTE:R_0402" H 3950 2800 50  0001 C CNN
@@
 $EndComp
 $Comp
-L Asiste:R_0402_10k R?
+L Asiste:R_0402_10k R402
 U 1 1 5B370CF9
 P 4250 3250
-F 0 "R?" H 4150 3400 50  0000 L CNN
+F 0 "R402" H 4150 3400 50  0000 L CNN
 F 1 "R_0402_10k" H 4250 2700 50  0001 C CNN
 F 2 "ASISTE:R_0402" H 4250 2800 50  0001 C CNN
@@
 $EndComp
 $Comp
-L Asiste:C_0402_100nF C?
+L Asiste:C_0402_100nF C401
 U 1 1 5B370D24
 P 5350 2950
-F 0 "C?" V 5300 2800 50  0000 L CNN
+F 0 "C401" V 5300 2800 50  0000 L CNN
 F 1 "C_0402_100nF" H 5100 2400 50  0001 L CNN
 F 2 "ASISTE:C_0402" H 5400 2700 50  0001 C CNN
@@
 $EndComp
 $Comp
-L Asiste:C_0402_100nF C?
+L Asiste:C_0402_100nF C402
 U 1 1 5B370E13
 P 6350 2950
-F 0 "C?" V 6300 2800 50  0000 L CNN
+F 0 "C402" V 6300 2800 50  0000 L CNN
 F 1 "C_0402_100nF" H 6100 2400 50  0001 L CNN
 F 2 "ASISTE:C_0402" H 6400 2700 50  0001 C CNN
@@
 	4250 3650 3850 3650
 $Comp
-L Asiste:MPU-6050 U?
+L Asiste:MPU-6050 U401
 U 1 1 5B56BC2F
 P 5850 3850
-F 0 "U?" H 5850 3064 50  0000 C CNN
+F 0 "U401" H 5850 3064 50  0000 C CNN
 F 1 "MPU-6050" H 5850 2973 50  0000 C CNN
 F 2 "ASISTE:QFN-24-1EP_4x4mm_Pitch0.5mm" H 5850 3050 50  0001 C CNN

Commit message: Añadido botón y otros
Parts:
- added R403: R_0402_100k, ASISTE:R_0402, symbol Asiste:R_0402_100k
Connections:
- wire segments 40 -> 44
Changed lines of the file:
@@
 $EndComp
 Connection ~ 5750 2950
-Text HLabel 6950 3550 2    60   Output ~ 0
+Text HLabel 7850 3550 2    60   Output ~ 0
 IMU_INT
 Wire Wire Line
-	6550 3550 6950 3550
+	6550 3550 7500 3550
 NoConn ~ 6550 3750
 NoConn ~ 6550 3850
@@
 	1    0    0    -1
 $EndComp
+$Comp
+L Asiste:R_0402_100k R403
+U 1 1 5B892CE4
+P 7500 3250
+F 0 "R403" H 7570 3296 50  0000 L CNN
+F 1 "R_0402_100k" H 7500 2700 50  0001 C CNN
+F 2 "ASISTE:R_0402" H 7500 2800 50  0001 C CNN
+F 3 "https://www.mouser.es/datasheet/2/427/rcge3-254226.pdf" H 7500 2900 50  0001 C CNN
+F 4 "RCG0402100KJNED" H 7450 3000 60  0001 C CNN "man#"
+F 5 "100k" H 7570 3205 50  0000 L CNN "Resistance"
+	1    7500 3250
+	1    0    0    -1
+$EndComp
+Wire Wire Line
+	7500 3400 7500 3550
+Connection ~ 7500 3550
+Wire Wire Line
+	7500 3550 7850 3550
+Wire Wire Line
+	7500 3100 7500 2650
+Wire Wire Line
+	7500 2650 5950 2650
+Connection ~ 5950 2650
 $EndSCHEMATC

Commit message: Esquemáticos totalmente terminados y revisados PCB a falta de routear el puerto de programación
Parts:
- removed C402: C_0402_100nF, ASISTE:C_0402, symbol Asiste:C_0402_100nF
- removed C404: C_0402_2.2nF, ASISTE:C_0402, symbol Asiste:C_0402_2.2nF
- added C11: C_0603_10nF, ASISTE:C_0603, symbol Asiste:C_0603_10nF
- added C13: C_0402_2.2nF, ASISTE:C_0402, symbol Asiste:C_0402_2.2nF
- renumbered C401 to C10, C403 to C12, R401 to R12, R402 to R13, R403 to R14, U401 to U3
Changed lines of the file:
@@
 $EndDescr
 $Comp
-L Asiste:GND #PWR0404
+L Asiste:GND #PWR025
 U 1 1 5B266BE2
 P 5850 4700
-F 0 "#PWR0404" H 5850 4450 50  0001 C CNN
+F 0 "#PWR025" H 5850 4450 50  0001 C CNN
 F 1 "GND" H 5850 4550 50  0000 C CNN
 F 2 "" H 5850 4700 50  0001 C CNN
@@
 AR Path="/5B266C17" Ref="#PWR?"  Part="1"
 AR Path="/5B26151D/5B266C17" Ref="#PWR?"  Part="1"
-AR Path="/5B56C4B2/5B266C17" Ref="#PWR0403"  Part="1"
-F 0 "#PWR0403" H 5850 2500 50  0001 C CNN
+AR Path="/5B56C4B2/5B266C17" Ref="#PWR024"  Part="1"
+F 0 "#PWR024" H 5850 2500 50  0001 C CNN
 F 1 "+3V3" H 5850 2790 50  0000 C CNN
 F 2 "" H 5850 2650 50  0001 C CNN
@@
 $EndComp
 $Comp
-L Asiste:GND #PWR0405
+L Asiste:GND #PWR026
 U 1 1 5B267277
 P 7000 3100
-F 0 "#PWR0405" H 7000 2850 50  0001 C CNN
+F 0 "#PWR026" H 7000 2850 50  0001 C CNN
 F 1 "GND" H 7000 2950 50  0000 C CNN
 F 2 "" H 7000 3100 50  0001 C CNN
@@
 	4600 2950 4600 3100
 $Comp
-L Asiste:GND #PWR0401
+L Asiste:GND #PWR022
 U 1 1 5B267478
 P 4600 3100
-F 0 "#PWR0401" H 4600 2850 50  0001 C CNN
+F 0 "#PWR022" H 4600 2850 50  0001 C CNN
 F 1 "GND" H 4600 2950 50  0000 C CNN
 F 2 "" H 4600 3100 50  0001 C CNN
@@
 	6950 4150 6550 4150
 $Comp
-L Asiste:GND #PWR0406
+L Asiste:GND #PWR027
 U 1 1 5B26785D
 P 7300 4700
-F 0 "#PWR0406" H 7300 4450 50  0001 C CNN
+F 0 "#PWR027" H 7300 4450 50  0001 C CNN
 F 1 "GND" H 7300 4550 50  0000 C CNN
 F 2 "" H 7300 4700 50  0001 C CNN
@@
 Connection ~ 7300 4650
 $Comp
-L Asiste:GND #PWR0402
+L Asiste:GND #PWR023
 U 1 1 5B2678F3
 P 4950 4200
-F 0 "#PWR0402" H 4950 3950 50  0001 C CNN
+F 0 "#PWR023" H 4950 3950 50  0001 C CNN
 F 1 "GND" H 4950 4050 50  0000 C CNN
 F 2 "" H 4950 4200 50  0001 C CNN
@@
 Connection ~ 4250 3650
 $Comp
-L Asiste:C_0402_2.2nF C404
-U 1 1 5B370B27
-P 7300 4400
-F 0 "C404" H 7325 4500 50  0000 L CNN
-F 1 "C_0402_2.2nF" H 7150 3850 50  0001 L CNN
-F 2 "ASISTE:C_0402" H 7350 4150 50  0001 C CNN
-F 3 "https://www.mouser.es/datasheet/2/445/885012205027-554116.pdf" H 7850 4050 50  0001 C CNN
-F 4 "885012205027" H 7300 3950 60  0001 C CNN "man#"
-F 5 "2.2nF" H 7350 4300 50  0000 L CNN "Capacitance"
-F 6 "16V" H 7250 3750 50  0001 L CNN "Voltage"
-	1    7300 4400
-	1    0    0    -1
-$EndComp
-$Comp
-L Asiste:C_0402_100nF C403
+L Asiste:C_0402_100nF C12
 U 1 1 5B370BA6
 P 6950 4400
-F 0 "C403" H 6975 4500 50  0000 L CNN
+F 0 "C12" H 6975 4500 50  0000 L CNN
 F 1 "C_0402_100nF" H 6700 3850 50  0001 L CNN
 F 2 "ASISTE:C_0402" H 7000 4150 50  0001 C CNN
@@
 $EndComp
 $Comp
-L Asiste:R_0402_10k R401
+L Asiste:R_0402_10k R12
 U 1 1 5B370C5C
 P 3950 3250
-F 0 "R401" H 3850 3400 50  0000 L CNN
+F 0 "R12" H 3750 3400 50  0000 L CNN
 F 1 "R_0402_10k" H 3950 2700 50  0001 C CNN
 F 2 "ASISTE:R_0402" H 3950 2800 50  0001 C CNN
@@
 $EndComp
 $Comp
-L Asiste:R_0402_10k R402
+L Asiste:R_0402_10k R13
 U 1 1 5B370CF9
 P 4250 3250
-F 0 "R402" H 4150 3400 50  0000 L CNN
+F 0 "R13" H 4050 3400 50  0000 L CNN
 F 1 "R_0402_10k" H 4250 2700 50  0001 C CNN
 F 2 "ASISTE:R_0402" H 4250 2800 50  0001 C CNN
@@
 $EndComp
 $Comp
-L Asiste:C_0402_100nF C401
+L Asiste:C_0402_100nF C10
 U 1 1 5B370D24
 P 5350 2950
-F 0 "C401" V 5300 2800 50  0000 L CNN
+F 0 "C10" V 5300 2650 50  0000 L CNN
 F 1 "C_0402_100nF" H 5100 2400 50  0001 L CNN
 F 2 "ASISTE:C_0402" H 5400 2700 50  0001 C CNN
@@
 	0    1    1    0
 $EndComp
-$Comp
-L Asiste:C_0402_100nF C402
-U 1 1 5B370E13
-P 6350 2950
-F 0 "C402" V 6300 2800 50  0000 L CNN
-F 1 "C_0402_100nF" H 6100 2400 50  0001 L CNN
-F 2 "ASISTE:C_0402" H 6400 2700 50  0001 C CNN
-F 3 "https://www.mouser.es/datasheet/2/281/murata_03122018_GCM_Series-1310150.pdf" H 6900 2600 50  0001 C CNN
-F 4 "GCM155R71C104KA55D" H 6350 2500 60  0001 C CNN "man#"
-F 5 "100nF" V 6300 3000 50  0000 L CNN "Capacitance"
-F 6 "16V" H 6300 2300 50  0001 L CNN "Voltage"
-	1    6350 2950
-	0    1    1    0
-$EndComp
 Wire Wire Line
 	5850 2650 5950 2650
@@
 	4250 3650 3850 3650
 $Comp
-L Asiste:MPU-6050 U401
+L Asiste:MPU-6050 U3
 U 1 1 5B56BC2F
 P 5850 3850
-F 0 "U401" H 5850 3064 50  0000 C CNN
-F 1 "MPU-6050" H 5850 2973 50  0000 C CNN
+F 0 "U3" H 5450 4400 50  0000 C CNN
+F 1 "MPU-6050" H 6200 4400 50  0000 C CNN
 F 2 "ASISTE:QFN-24-1EP_4x4mm_Pitch0.5mm" H 5850 3050 50  0001 C CNN
 F 3 "https://www.invensense.com/wp-content/uploads/2015/02/MPU-6000-Datasheet1.pdf" H 5900 2900 50  0001 C CNN
@@
 $EndComp
 $Comp
-L Asiste:R_0402_100k R403
+L Asiste:R_0402_100k R14
 U 1 1 5B892CE4
 P 7500 3250
-F 0 "R403" H 7570 3296 50  0000 L CNN
+F 0 "R14" H 7570 3296 50  0000 L CNN
 F 1 "R_0402_100k" H 7500 2700 50  0001 C CNN
 F 2 "ASISTE:R_0402" H 7500 2800 50  0001 C CNN
@@
 	7500 2650 5950 2650
 Connection ~ 5950 2650
+$Comp
+L Asiste:C_0402_2.2nF C13
+U 1 1 5B97D3AF
+P 7300 4400
+F 0 "C13" H 7400 4500 50  0000 L CNN
+F 1 "C_0402_2.2nF" H 7150 3850 50  0001 L CNN
+F 2 "ASISTE:C_0402" H 7350 4150 50  0001 C CNN
+F 3 "https://www.mouser.es/datasheet/2/445/885012205027-554116.pdf" H 7850 4050 50  0001 C CNN
+F 4 "GCM155R71H222KA37D" H 7300 3950 60  0001 C CNN "man#"
+F 5 "2.2nF" H 7400 4300 50  0000 L CNN "Capacitance"
+F 6 "50V" H 7250 3750 50  0001 L CNN "Voltage"
+	1    7300 4400
+	1    0    0    -1
+$EndComp
+$Comp
+L Asiste:C_0603_10nF C11
+U 1 1 5B95104D
+P 6350 2950
+F 0 "C11" V 6300 2800 50  0000 C CNN
+F 1 "C_0603_10nF" H 6100 2300 50  0001 L CNN
+F 2 "ASISTE:C_0603" H 6400 2700 50  0001 C CNN
+F 3 "https://www.mouser.es/datasheet/2/400/lcc_commercial_general_en-837201.pdf" H 6900 2600 50  0001 C CNN
+F 4 "C0603X7R0J103M030BC" H 6350 2400 60  0001 C CNN "man#"
+F 5 "10nF" V 6300 3100 50  0000 C CNN "Capacitance"
+F 6 "6.3V" H 6350 2500 60  0001 C CNN "Voltage"
+	1    6350 2950
+	0    1    1    0
+$EndComp
 $EndSCHEMATC

Commit message: Actualizando
Parts:
- renumbered C11 to C10, C12 to C11, C13 to C12, C10 to C9
Changed lines of the file:
@@
 Connection ~ 4250 3650
 $Comp
-L Asiste:C_0402_100nF C12
+L Asiste:C_0402_100nF C11
 U 1 1 5B370BA6
 P 6950 4400
-F 0 "C12" H 6975 4500 50  0000 L CNN
+F 0 "C11" H 6975 4500 50  0000 L CNN
 F 1 "C_0402_100nF" H 6700 3850 50  0001 L CNN
 F 2 "ASISTE:C_0402" H 7000 4150 50  0001 C CNN
@@
 $EndComp
 $Comp
-L Asiste:C_0402_100nF C10
+L Asiste:C_0402_100nF C9
 U 1 1 5B370D24
 P 5350 2950
-F 0 "C10" V 5300 2650 50  0000 L CNN
+F 0 "C9" V 5300 2650 50  0000 L CNN
 F 1 "C_0402_100nF" H 5100 2400 50  0001 L CNN
 F 2 "ASISTE:C_0402" H 5400 2700 50  0001 C CNN
@@
 Connection ~ 5950 2650
 $Comp
-L Asiste:C_0402_2.2nF C13
+L Asiste:C_0402_2.2nF C12
 U 1 1 5B97D3AF
 P 7300 4400
-F 0 "C13" H 7400 4500 50  0000 L CNN
+F 0 "C12" H 7400 4500 50  0000 L CNN
 F 1 "C_0402_2.2nF" H 7150 3850 50  0001 L CNN
 F 2 "ASISTE:C_0402" H 7350 4150 50  0001 C CNN
@@
 $EndComp
 $Comp
-L Asiste:C_0603_10nF C11
+L Asiste:C_0603_10nF C10
 U 1 1 5B95104D
 P 6350 2950
-F 0 "C11" V 6300 2800 50  0000 C CNN
+F 0 "C10" V 6300 2800 50  0000 C CNN
 F 1 "C_0603_10nF" H 6100 2300 50  0001 L CNN
 F 2 "ASISTE:C_0603" H 6400 2700 50  0001 C CNN
