File: micro.sch (KiCad schematic (older format))
At the start: 23 parts

Commit message: Terminado esquemático. Falta revisar
Parts:
- removed AE?: Antenna_Chip, symbol Asiste:Antenna_Chip
- removed C?: C_0402_2.2pF, ASISTE:C_0402, symbol Asiste:C_0402_2.2pF
- removed C?: C_0402_1pF, ASISTE:C_0402, symbol Asiste:C_0402_1pF
- removed C?: C_0402_1.5pF, ASISTE:C_0402, symbol Asiste:C_0402_1.5pF
- removed L?: L_0402_4.7nH, ASISTE:L_0402, symbol Asiste:L_0402_4.7nH
- removed L?: L_0603_10nH, ASISTE:L_0603, symbol Asiste:L_0603_10nH
- removed L?: L_0402_3.3nH, ASISTE:L_0402, symbol Asiste:L_0402_3.3nH
- added AE?: Antenna_Chip, ASISTE:ANT, symbol Asiste:Antenna_Chip
- added ANT?: 2450BM14E0003, ASISTE:BALUN-2450BM14E0003, symbol Asiste:2450BM14E0003
- added C?: C_0402_1.2pF, ASISTE:C_0402, symbol Asiste:C_0402_1.2pF
- added L?: L_0402_2.7nH, ASISTE:L_0402, symbol Asiste:L_0402_2.7nH
- added L?: L_0402_3.3nH, ASISTE:L_0402, symbol Asiste:L_0402_3.3nH
Connections:
- net labels added: BAT_CHG_STAT, BUTTON, PWR_EN
- wire segments 114 -> 119
- no-connect marks 17 -> 14

Commit message: Esquemático parcialmente revisado. Falta revisar pines y correspondencia con footprints
Parts:
- removed U?: nRF51x22-QFxx, Package_DFN_QFN:QFN-48-1EP_6x6mm_P0.4mm_EP4.66x4.66mm, symbol Asiste:nRF51x22-QFxx
- added C511, C512: C_0402_12pF, ASISTE:C_0402, symbol Asiste:C_0402_12pF
- added U501: nRF51x22-QFxx, ASISTE:QFN-48-1EP_6x6mm_Pitch0.4mm_ThermalVias, symbol Asiste:nRF51x22-QFxx
- added Y502: Crystal_3.2x1.5, ASISTE:Crystal_SMD_G8-2Pin_3.2x1.5mm, symbol Asiste:Crystal_3.2x1.5
- gave numbers to parts that had none: 20
Connections:
- net labels added: BAT_SENSE, HR_~INT, IMU_INT, IMU_SCL, IMU_SDA, TMP_ALERT
- net labels removed: MCU_AN1, MCU_INT2, MCU_INT3, MCU_PROG_~CTS, MCU_PROG_~RTS, MPU_INT1, MPU_SCL1, MPU_SDA1
- wire segments 119 -> 128

Commit message: Añadido botón y otros
Parts:
- renumbered AE501 to AE601, ANT501 to ANT601, C501 to C601, C502 to C602, C503 to C603, C504 to C604, C505 to C605, C506 to C606, C507 to C607, C508 to C608, C509 to C609, C510 to C610, C511 to C611, C512 to C612, L501 to L601, L502 to L602, L503 to L603, L504 to L604, R502 to R601, R503 to R602, R501 to R603, U501 to U601, Y501 to Y601, Y502 to Y602

Commit message: Esquemáticos totalmente terminados y revisados PCB a falta de routear el puerto de programación
Parts:
- removed ANT601: 2450BM14E0003, ASISTE:BALUN-2450BM14E0003, symbol Asiste:2450BM14E0003
- removed C601: C_0402_1.2pF, ASISTE:C_0402, symbol Asiste:C_0402_1.2pF
- removed L601: L_0402_3.3nH, ASISTE:L_0402, symbol Asiste:L_0402_3.3nH
- removed L602: L_0402_2.7nH, ASISTE:L_0402, symbol Asiste:L_0402_2.7nH
- added C15: C_0402_1.5pF, ASISTE:C_0402, symbol Asiste:C_0402_1.5pF
- added C18: C_0402_1pF, ASISTE:C_0402, symbol Asiste:C_0402_1pF
- added C19: C_0402_2.2pF, ASISTE:C_0402, symbol Asiste:C_0402_2.2pF
- added L1: L_0402_3.3nH, ASISTE:L_0402, symbol Asiste:L_0402_3.3nH
- added L2: L_0603_10nH, ASISTE:L_0603, symbol Asiste:L_0603_10nH
- added L3: L_0402_4.7nH, ASISTE:L_0402, symbol Asiste:L_0402_4.7nH
- renumbered AE601 to AE1, C602 to C16, C603 to C17, C604 to C20, C605 to C21, C606 to C22, C607 to C23, C608 to C24, C609 to C25, C610 to C26, C611 to C27, C612 to C28, L603 to L4, L604 to L5, R601 to R16, R602 to R17, R603 to R18, U601 to U5, Y601 to Y1, Y602 to Y2
Connections:
- net labels removed: PWR_EN
- wire segments 128 -> 130
- no-connect marks 14 -> 15

Commit message: Actualizando
Parts:
- renumbered C15 to C14, C16 to C15, C17 to C16, C18 to C17, C19 to C18, C20 to C19, C21 to C20, C22 to C21, C23 to C22, C24 to C23, C25 to C24, C26 to C25, C27 to C26, C28 to C27
Connections:
- net labels added: MCU_PROG_RX
- net labels removed: MPU_PROG_RX
Changed lines of the file:
@@
 $EndComp
 $Comp
-L Asiste:C_0402_12pF C16
+L Asiste:C_0402_12pF C15
 U 1 1 5B370614
 P 3350 4400
-F 0 "C16" V 3250 4250 50  0000 L CNN
+F 0 "C15" V 3250 4250 50  0000 L CNN
 F 1 "C_0402_12pF" H 3100 3850 50  0001 L CNN
 F 2 "ASISTE:C_0402" H 3400 4150 50  0001 C CNN
@@
 $EndComp
 $Comp
-L Asiste:C_0402_12pF C17
+L Asiste:C_0402_12pF C16
 U 1 1 5B3706F1
 P 3350 5150
-F 0 "C17" V 3250 5000 50  0000 L CNN
+F 0 "C16" V 3250 5000 50  0000 L CNN
 F 1 "C_0402_12pF" H 3100 4600 50  0001 L CNN
 F 2 "ASISTE:C_0402" H 3400 4900 50  0001 C CNN
@@
 $EndComp
 $Comp
-L Asiste:C_0402_100nF C25
+L Asiste:C_0402_100nF C24
 U 1 1 5B37082F
 P 5100 2100
-F 0 "C25" V 5050 1850 50  0000 L CNN
+F 0 "C24" V 5050 1850 50  0000 L CNN
 F 1 "C_0402_100nF" H 4850 1550 50  0001 L CNN
 F 2 "ASISTE:C_0402" H 5150 1850 50  0001 C CNN
@@
 $EndComp
 $Comp
-L Asiste:C_0402_47nF C24
+L Asiste:C_0402_47nF C23
 U 1 1 5B3708DB
 P 5100 1850
-F 0 "C24" V 5050 1600 50  0000 L CNN
+F 0 "C23" V 5050 1600 50  0000 L CNN
 F 1 "C_0402_47nF" H 4900 1300 50  0001 L CNN
 F 2 "ASISTE:C_0402" H 5150 1600 50  0001 C CNN
@@
 $EndComp
 $Comp
-L Asiste:C_0603_1uF C26
+L Asiste:C_0603_1uF C25
 U 1 1 5B371645
 P 7850 2500
-F 0 "C26" V 7700 2400 50  0000 L CNN
+F 0 "C25" V 7700 2400 50  0000 L CNN
 F 1 "C_0603_1uF" H 7650 1950 50  0001 L CNN
 F 2 "ASISTE:C_0603" H 7900 2250 50  0001 C CNN
@@
 $EndComp
 $Comp
-L Asiste:C_0402_1nF C21
+L Asiste:C_0402_1nF C20
 U 1 1 5B371AE1
 P 5100 1100
-F 0 "C21" V 5050 850 50  0000 L CNN
+F 0 "C20" V 5050 850 50  0000 L CNN
 F 1 "C_0402_1nF" H 4900 550 50  0001 L CNN
 F 2 "ASISTE:C_0402" H 5150 850 50  0001 C CNN
@@
 $EndComp
 $Comp
-L Asiste:C_0603_4.7uF C23
+L Asiste:C_0603_4.7uF C22
 U 1 1 5B371CAF
 P 5100 1600
-F 0 "C23" V 5050 1350 50  0000 L CNN
+F 0 "C22" V 5050 1350 50  0000 L CNN
 F 1 "C_0603_4.7uF" H 4900 1050 50  0001 L CNN
 F 2 "ASISTE:C_0603" H 5150 1350 50  0001 C CNN
@@
 $EndComp
 $Comp
-L Asiste:C_0402_100nF C22
+L Asiste:C_0402_100nF C21
 U 1 1 5B372252
 P 5100 1350
-F 0 "C22" V 5050 1100 50  0000 L CNN
+F 0 "C21" V 5050 1100 50  0000 L CNN
 F 1 "C_0402_100nF" H 4850 800 50  0001 L CNN
 F 2 "ASISTE:C_0402" H 5150 1100 50  0001 C CNN
@@
 	7050 4050 7400 4050
 Text HLabel 7400 3850 2    60   Input ~ 0
-MPU_PROG_RX
+MCU_PROG_RX
 Text HLabel 7400 4050 2    60   Input ~ 0
 MCU_PROG_TX
@@
 	5600 2100 5600 2650
 $Comp
-L Asiste:C_0402_2.2nF C20
+L Asiste:C_0402_2.2nF C19
 U 1 1 5B64281A
 P 4100 2550
-F 0 "C20" V 3848 2550 50  0000 C CNN
+F 0 "C19" V 3848 2550 50  0000 C CNN
 F 1 "C_0402_2.2nF" H 3950 2000 50  0001 L CNN
 F 2 "ASISTE:C_0402" H 4150 2300 50  0001 C CNN
@@
 	7350 5850 8050 5850
 $Comp
-L Asiste:C_0402_12pF C27
+L Asiste:C_0402_12pF C26
 U 1 1 5B8D26A3
 P 8450 5550
-F 0 "C27" V 8198 5550 50  0000 C CNN
+F 0 "C26" V 8198 5550 50  0000 C CNN
 F 1 "C_0402_12pF" H 8200 5000 50  0001 L CNN
 F 2 "ASISTE:C_0402" H 8500 5300 50  0001 C CNN
@@
 $EndComp
 $Comp
-L Asiste:C_0402_12pF C28
+L Asiste:C_0402_12pF C27
 U 1 1 5B8D285F
 P 8450 5850
-F 0 "C28" V 8610 5850 50  0000 C CNN
+F 0 "C27" V 8610 5850 50  0000 C CNN
 F 1 "C_0402_12pF" H 8200 5300 50  0001 L CNN
 F 2 "ASISTE:C_0402" H 8500 5600 50  0001 C CNN
@@
 	4450 3100 4450 3250
 $Comp
-L Asiste:C_0402_2.2pF C19
+L Asiste:C_0402_2.2pF C18
 U 1 1 5B91A640
 P 3950 3600
-F 0 "C19" V 4250 3600 50  0000 C CNN
+F 0 "C18" V 4250 3600 50  0000 C CNN
 F 1 "C_0402_2.2pF" H 3750 3050 50  0001 L CNN
 F 2 "ASISTE:C_0402" H 4000 3350 50  0001 C CNN
@@
 Connection ~ 4450 3600
 $Comp
-L Asiste:C_0402_1pF C18
+L Asiste:C_0402_1pF C17
 U 1 1 5B941B9D
 P 3500 3800
-F 0 "C18" H 3350 3750 50  0000 R CNN
+F 0 "C17" H 3350 3750 50  0000 R CNN
 F 1 "C_0402_1pF" H 3300 3250 50  0001 L CNN
 F 2 "ASISTE:C_0402" H 3550 3550 50  0001 C CNN
@@
 $EndComp
 $Comp
-L Asiste:C_0402_1.5pF C15
+L Asiste:C_0402_1.5pF C14
 U 1 1 5B946038
 P 2800 3800
-F 0 "C15" H 2950 3850 50  0000 L CNN
+F 0 "C14" H 2950 3850 50  0000 L CNN
 F 1 "C_0402_1.5pF" H 2600 3250 50  0001 L CNN
 F 2 "ASISTE:C_0402" H 2850 3550 50  0001 C CNN
