File: power.sch (KiCad schematic (older format))
At the start: 8 parts

Commit message: Terminado esquemático. Falta revisar
Parts:
- added C? (x4): C_0603_1uF, ASISTE:C_0603, symbol Asiste:C_0603_1uF
- added D?: D_Schottky, ASISTE:D_SOD-123, symbol Asiste:D_Schottky
- added Q?: DMP1045U, ASISTE:SOT-23, symbol Asiste:DMP1045U
- added R?: R_0402_100k, ASISTE:R_0402, symbol Asiste:R_0402_100k
- added U?: XC6415CC91MR-G, ASISTE:TSOT-23-6, symbol Asiste:XC6415CC91MR-G
Connections:
- net labels added: +1V8, +3V3, PWR_EN, VCC
- wire segments 41 -> 80

Commit message: Esquemático parcialmente revisado. Falta revisar pines y correspondencia con footprints
Parts:
- removed U?: MCP73831, Package_TO_SOT_SMD:SOT-23-5, symbol Asiste:MCP73831
- added U301: MCP73831, ASISTE:TSOT-23-5, symbol Asiste:MCP73831
- gave numbers to parts that had none: 15
Connections:
- wire segments 80 -> 76
Changed lines of the file:
@@
 $EndDescr
 $Comp
-L Asiste:GND #PWR?
+L Asiste:GND #PWR0301
 U 1 1 5B69D268
 P 3200 5500
-F 0 "#PWR?" H 3200 5250 50  0001 C CNN
+F 0 "#PWR0301" H 3200 5250 50  0001 C CNN
 F 1 "GND" H 3205 5327 50  0000 C CNN
 F 2 "" H 3200 5500 50  0001 C CNN
@@
 $EndComp
 $Comp
-L Asiste:USB_B_Micro J?
+L Asiste:USB_B_Micro J301
 U 1 1 5B752AC5
 P 3200 5000
-F 0 "J?" H 3255 5467 50  0000 C CNN
+F 0 "J301" H 3255 5467 50  0000 C CNN
 F 1 "USB_B_Micro" H 3255 5376 50  0000 C CNN
 F 2 "ASISTE:USB_Micro-B_Molex-105017-0001" H 3150 4250 50  0001 C CNN
@@
 	3200 5450 3200 5500
 $Comp
-L Asiste:MCP73831 U?
-U 1 1 5B744957
-P 3900 3000
-F 0 "U?" H 3650 3250 50  0000 C CNN
-F 1 "MCP73831" H 4200 3250 50  0000 C CNN
-F 2 "Package_TO_SOT_SMD:SOT-23-5" H 3400 2250 50  0001 L CIN
-F 3 "http://ww1.microchip.com/downloads/en/DeviceDoc/20001984g.pdf" H 3900 2350 50  0001 C CNN
-F 4 "MCP73831T-2ACI/OT" H 3900 3650 60  0001 C CNN "man#"
-	1    3900 3000
-	1    0    0    -1
-$EndComp
-$Comp
-L Asiste:GND #PWR?
+L Asiste:GND #PWR0304
 U 1 1 5B744A7C
 P 3900 3550
-F 0 "#PWR?" H 3900 3300 50  0001 C CNN
+F 0 "#PWR0304" H 3900 3300 50  0001 C CNN
 F 1 "GND" H 3905 3377 50  0000 C CNN
 F 2 "" H 3900 3550 50  0001 C CNN
@@
 	3900 2550 3900 2600
 $Comp
-L Asiste:VBAT #PWR?
+L Asiste:VBAT #PWR0305
 U 1 1 5B7453C9
 P 5300 2600
-F 0 "#PWR?" H 5300 2450 50  0001 C CNN
+F 0 "#PWR0305" H 5300 2450 50  0001 C CNN
 F 1 "VBAT" H 5315 2773 50  0000 C CNN
 F 2 "" H 5300 2600 50  0001 C CNN
@@
 	3900 3500 3900 3550
 $Comp
-L Asiste:C_0603_4.7uF C?
+L Asiste:C_0603_4.7uF C301
 U 1 1 5B745D35
 P 2650 3050
-F 0 "C?" H 2536 3004 50  0000 R CNN
+F 0 "C301" H 2536 3004 50  0000 R CNN
 F 1 "C_0603_4.7uF" H 2450 2500 50  0001 L CNN
 F 2 "ASISTE:C_0603" H 2700 2800 50  0001 C CNN
@@
 Connection ~ 3300 3500
 $Comp
-L Asiste:C_0603_4.7uF C?
+L Asiste:C_0603_4.7uF C302
 U 1 1 5B74635C
 P 5300 3050
-F 0 "C?" H 5415 3096 50  0000 L CNN
+F 0 "C302" H 5415 3096 50  0000 L CNN
 F 1 "C_0603_4.7uF" H 5100 2500 50  0001 L CNN
 F 2 "ASISTE:C_0603" H 5350 2800 50  0001 C CNN
@@
 	4550 2600 5300 2600
 Wire Wire Line
-	4550 2600 4550 2900
-Wire Wire Line
 	5300 2600 5300 2900
 Connection ~ 5300 2600
@@
 	4300 3100 4400 3100
 $Comp
-L Asiste:PWR_FLAG #FLG?
-U 1 1 5B748A67
-P 3950 4750
-F 0 "#FLG?" H 3950 4825 50  0001 C CNN
-F 1 "PWR_FLAG" H 3950 4924 50  0000 C CNN
-F 2 "" H 3950 4750 50  0001 C CNN
-F 3 "~" H 3950 4750 50  0001 C CNN
-	1    3950 4750
-	1    0    0    -1
-$EndComp
-Wire Wire Line
-	3600 4800 3950 4800
-Wire Wire Line
-	3950 4800 3950 4750
-Connection ~ 3600 4800
-$Comp
-L Asiste:PWR_FLAG #FLG?
-U 1 1 5B749035
-P 3550 5500
-F 0 "#FLG?" H 3550 5575 50  0001 C CNN
-F 1 "PWR_FLAG" H 3550 5673 50  0000 C CNN
-F 2 "" H 3550 5500 50  0001 C CNN
-F 3 "~" H 3550 5500 50  0001 C CNN
-	1    3550 5500
-	-1   0    0    1
-$EndComp
-Wire Wire Line
-	3200 5450 3550 5450
-Wire Wire Line
-	3550 5450 3550 5500
-$Comp
-L Asiste:PWR_FLAG #FLG?
-U 1 1 5B749B97
-P 2650 2550
-F 0 "#FLG?" H 2650 2625 50  0001 C CNN
-F 1 "PWR_FLAG" H 2650 2724 50  0000 C CNN
-F 2 "" H 2650 2550 50  0001 C CNN
-F 3 "~" H 2650 2550 50  0001 C CNN
-	1    2650 2550
-	1    0    0    -1
-$EndComp
-Wire Wire Line
-	2650 2550 2650 2600
-Connection ~ 2650 2600
-$Comp
-L Asiste:PWR_FLAG #FLG?
-U 1 1 5B74A256
-P 4550 2550
-F 0 "#FLG?" H 4550 2625 50  0001 C CNN
-F 1 "PWR_FLAG" H 4550 2724 50  0000 C CNN
-F 2 "" H 4550 2550 50  0001 C CNN
-F 3 "~" H 4550 2550 50  0001 C CNN
-	1    4550 2550
-	1    0    0    -1
-$EndComp
-Wire Wire Line
-	4550 2600 4550 2550
-Connection ~ 4550 2600
-$Comp
-L Asiste:R_0402_2k R?
+L Asiste:R_0402_2k R301
 U 1 1 5B74B4B5
 P 3300 3300
-F 0 "R?" H 3370 3346 50  0000 L CNN
+F 0 "R301" H 3370 3346 50  0000 L CNN
 F 1 "R_0402_2k" H 3300 2750 50  0001 C CNN
 F 2 "ASISTE:R_0402" H 3300 2850 50  0001 C CNN
@@
 $EndComp
 $Comp
-L Asiste:R_0402_2M2 R?
+L Asiste:R_0402_2M2 R303
 U 1 1 5B74D1E7
 P 5900 3250
-F 0 "R?" H 5970 3296 50  0000 L CNN
+F 0 "R303" H 5970 3296 50  0000 L CNN
 F 1 "R_0402_2M2" H 5900 2700 50  0001 C CNN
 F 2 "ASISTE:R_0402" H 5900 2800 50  0001 C CNN
@@
 $EndComp
 $Comp
-L Asiste:R_0402_10M R?
+L Asiste:R_0402_10M R302
 U 1 1 5B74D9F6
 P 5900 2850
-F 0 "R?" H 5970 2896 50  0000 L CNN
+F 0 "R302" H 5970 2896 50  0000 L CNN
 F 1 "R_0402_10M" H 5900 2300 50  0001 C CNN
 F 2 "ASISTE:R_0402" H 5900 2400 50  0001 C CNN
@@
 BAT_SENSE
 $Comp
-L Asiste:VBUS #PWR?
+L Asiste:VBUS #PWR0302
 U 1 1 5B795544
 P 3600 4700
-F 0 "#PWR?" H 3600 4550 50  0001 C CNN
+F 0 "#PWR0302" H 3600 4550 50  0001 C CNN
 F 1 "VBUS" H 3615 4873 50  0000 C CNN
 F 2 "" H 3600 4700 50  0001 C CNN
@@
 $EndComp
 $Comp
-L Asiste:VBUS #PWR?
+L Asiste:VBUS #PWR0303
 U 1 1 5B7955CD
 P 3900 2550
-F 0 "#PWR?" H 3900 2400 50  0001 C CNN
+F 0 "#PWR0303" H 3900 2400 50  0001 C CNN
 F 1 "VBUS" H 3915 2723 50  0000 C CNN
 F 2 "" H 3900 2550 50  0001 C CNN
@@
 	2300 6900 1100 6900
 $Comp
-L Asiste:Conn_01x02 J?
+L Asiste:Conn_01x02 J302
 U 1 1 5B79A067
 P 7450 2600
-F 0 "J?" H 7530 2592 50  0000 L CNN
+F 0 "J302" H 7530 2592 50  0000 L CNN
 F 1 "Conn_01x02" H 7530 2501 50  0000 L CNN
 F 2 "ASISTE:JST_SH_SM02B-SRSS-TB_1x02-1MP_P1.00mm_Horizontal" H 7500 2100 50  0001 C CNN
@@
 Connection ~ 5900 3500
 $Comp
-L Asiste:DMP1045U Q?
+L Asiste:DMP1045U Q301
 U 1 1 5B86EC1C
 P 7950 1900
-F 0 "Q?" V 8200 1900 50  0000 C CNN
+F 0 "Q301" V 8200 1900 50  0000 C CNN
 F 1 "DMP1045U" V 8291 1900 50  0000 C CNN
 F 2 "ASISTE:SOT-23" H 8050 1400 50  0001 C CNN
@@
 	3150 2600 3900 2600
 $Comp
-L Asiste:D_Schottky D?
+L Asiste:D_Schottky D301
 U 1 1 5B8728BF
 P 8700 1750
-F 0 "D?" V 8746 1671 50  0000 R CNN
+F 0 "D301" V 8746 1671 50  0000 R CNN
 F 1 "D_Schottky" V 8655 1671 50  0000 R CNN
 F 2 "ASISTE:D_SOD-123" H 8700 1350 50  0001 C CNN
@@
 	8700 2000 8700 1900
 $Comp
-L Asiste:C_0603_1uF C?
+L Asiste:C_0603_1uF C306
 U 1 1 5B875437
 P 8700 3050
-F 0 "C?" H 8815 3096 50  0000 L CNN
+F 0 "C306" H 8815 3096 50  0000 L CNN
 F 1 "C_0603_1uF" H 8500 2500 50  0001 L CNN
 F 2 "ASISTE:C_0603" H 8750 2800 50  0001 C CNN
@@
 Connection ~ 7250 3500
 $Comp
-L Asiste:R_0402_100k R?
+L Asiste:R_0402_100k R304
 U 1 1 5B87AE63
 P 9500 2500
-F 0 "R?" H 9570 2546 50  0000 L CNN
+F 0 "R304" H 9570 2546 50  0000 L CNN
 F 1 "R_0402_100k" H 9500 1950 50  0001 C CNN
 F 2 "ASISTE:R_0402" H 9500 2050 50  0001 C CNN
@@
 Connection ~ 8700 3500
 $Comp
-L Asiste:VCC #PWR?
+L Asiste:VCC #PWR0310
 U 1 1 5B882208
 P 8800 2000
-F 0 "#PWR?" H 8800 1850 50  0001 C CNN
+F 0 "#PWR0310" H 8800 1850 50  0001 C CNN
 F 1 "VCC" V 8815 2128 50  0000 L CNN
 F 2 "" H 8800 2000 50  0001 C CNN
@@
 	8700 2000 8800 2000
 $Comp
-L Asiste:XC6415CC91MR-G U?
+L Asiste:XC6415CC91MR-G U302
 U 1 1 5B890199
 P 7350 5000
-F 0 "U?" H 7050 5200 60  0000 C CNN
+F 0 "U302" H 7050 5200 60  0000 C CNN
 F 1 "XC6415CC91MR-G" H 7850 5200 60  0000 C CNN
 F 2 "ASISTE:TSOT-23-6" H 6950 5100 60  0001 C CNN
@@
 $EndComp
 $Comp
-L Asiste:VCC #PWR?
+L Asiste:VCC #PWR0306
 U 1 1 5B890448
 P 7350 4600
-F 0 "#PWR?" H 7350 4450 50  0001 C CNN
+F 0 "#PWR0306" H 7350 4450 50  0001 C CNN
 F 1 "VCC" H 7365 4773 50  0000 C CNN
 F 2 "" H 7350 4600 50  0001 C CNN
@@
 	7350 4600 7350 4650
 $Comp
-L Asiste:GND #PWR?
+L Asiste:GND #PWR0307
 U 1 1 5B8910DA
 P 7350 5750
-F 0 "#PWR?" H 7350 5500 50  0001 C CNN
+F 0 "#PWR0307" H 7350 5500 50  0001 C CNN
 F 1 "GND" H 7355 5577 50  0000 C CNN
 F 2 "" H 7350 5750 50  0001 C CNN
@@
 	7800 4950 8500 4950
 $Comp
-L Asiste:C_0603_1uF C?
+L Asiste:C_0603_1uF C305
 U 1 1 5B89B89A
 P 8500 5450
-F 0 "C?" H 8615 5496 50  0000 L CNN
+F 0 "C305" H 8615 5496 50  0000 L CNN
 F 1 "C_0603_1uF" H 8300 4900 50  0001 L CNN
 F 2 "ASISTE:C_0603" H 8550 5200 50  0001 C CNN
@@
 $EndComp
 $Comp
-L Asiste:C_0603_1uF C?
+L Asiste:C_0603_1uF C304
 U 1 1 5B89B95E
 P 7950 5450
-F 0 "C?" H 8065 5496 50  0000 L CNN
+F 0 "C304" H 8065 5496 50  0000 L CNN
 F 1 "C_0603_1uF" H 7750 4900 50  0001 L CNN
 F 2 "ASISTE:C_0603" H 8000 5200 50  0001 C CNN
@@
 Connection ~ 8500 4950
 $Comp
-L Asiste:C_0603_1uF C?
+L Asiste:C_0603_1uF C303
 U 1 1 5B8A2E24
 P 6800 5450
-F 0 "C?" H 6915 5496 50  0000 L CNN
+F 0 "C303" H 6915 5496 50  0000 L CNN
 F 1 "C_0603_1uF" H 6600 4900 50  0001 L CNN
 F 2 "ASISTE:C_0603" H 6850 5200 50  0001 C CNN
@@
 	6800 5700 7350 5700
 $Comp
-L Asiste:+1V8 #PWR?
+L Asiste:+1V8 #PWR0309
 U 1 1 5B8AB235
 P 8500 4850
-F 0 "#PWR?" H 8500 4700 50  0001 C CNN
+F 0 "#PWR0309" H 8500 4700 50  0001 C CNN
 F 1 "+1V8" H 8650 4900 50  0000 C CNN
 F 2 "" H 8500 4850 50  0001 C CNN
@@
 $EndComp
 $Comp
-L Asiste:+3V3 #PWR?
+L Asiste:+3V3 #PWR0308
 U 1 1 5B8AB308
 P 7950 5150
-F 0 "#PWR?" H 7950 5000 50  0001 C CNN
+F 0 "#PWR0308" H 7950 5000 50  0001 C CNN
 F 1 "+3V3" H 8100 5200 50  0000 C CNN
 F 2 "" H 7950 5150 50  0001 C CNN
@@
 Wire Wire Line
 	6800 4650 6800 5200
+$Comp
+L Asiste:PWR_FLAG #FLG0301
+U 1 1 5B8BB2C5
+P 7650 4600
+F 0 "#FLG0301" H 7650 4675 50  0001 C CNN
+F 1 "PWR_FLAG" H 7650 4774 50  0000 C CNN
+F 2 "" H 7650 4600 50  0001 C CNN
+F 3 "~" H 7650 4600 50  0001 C CNN
+	1    7650 4600
+	1    0    0    -1
+$EndComp
+Wire Wire Line
+	7350 4650 7650 4650
+Wire Wire Line
+	7650 4650 7650 4600
+Wire Wire Line
+	4550 2600 4550 2900
+$Comp
+L Asiste:MCP73831 U301
+U 1 1 5B8C4CF4
+P 3900 3000
+F 0 "U301" H 3650 3250 50  0000 C CNN
+F 1 "MCP73831" H 4150 3250 50  0000 C CNN
+F 2 "ASISTE:TSOT-23-5" H 3400 2250 50  0001 L CIN
+F 3 "http://ww1.microchip.com/downloads/en/DeviceDoc/20001984g.pdf" H 3900 2350 50  0001 C CNN
+F 4 "MCP73831T-2ACI/OT" H 3900 3650 60  0001 C CNN "man#"
+	1    3900 3000
+	1    0    0    -1
+$EndComp
 $EndSCHEMATC

Commit message: Esquemáticos totalmente terminados y revisados PCB a falta de routear el puerto de programación
Parts:
- removed J301: USB_B_Micro, ASISTE:USB_Micro-B_Molex-105017-0001, symbol Asiste:USB_B_Micro
- added J1: USB_B_Micro_SMD, ASISTE:USB_Micro-B_Molex_47346-0001, symbol Asiste:USB_B_Micro_SMD
- renumbered C301 to C4, C302 to C5, C303 to C6, C304 to C7, C305 to C8, C306 to C9, D301 to D2, J302 to J2, Q301 to Q4, R303 to R10, R304 to R11, R301 to R8, R302 to R9, U301 to U1, U302 to U2
Connections:
- net labels removed: PWR_EN
- wire segments 76 -> 77
Changed lines of the file:
@@
 $EndDescr
 $Comp
-L Asiste:GND #PWR0301
+L Asiste:GND #PWR012
 U 1 1 5B69D268
 P 3200 5500
-F 0 "#PWR0301" H 3200 5250 50  0001 C CNN
+F 0 "#PWR012" H 3200 5250 50  0001 C CNN
 F 1 "GND" H 3205 5327 50  0000 C CNN
 F 2 "" H 3200 5500 50  0001 C CNN
@@
 	1    0    0    -1
 $EndComp
-$Comp
-L Asiste:USB_B_Micro J301
-U 1 1 5B752AC5
-P 3200 5000
-F 0 "J301" H 3255 5467 50  0000 C CNN
-F 1 "USB_B_Micro" H 3255 5376 50  0000 C CNN
-F 2 "ASISTE:USB_Micro-B_Molex-105017-0001" H 3150 4250 50  0001 C CNN
-F 3 "https://www.mouser.es/datasheet/2/276/1050170001_IO_CONNECTORS-230168.pdf" H 3250 4150 50  0001 C CNN
-F 4 "105017-0001" H 3200 4050 60  0001 C CNN "man#"
-	1    3200 5000
-	1    0    0    -1
-$EndComp
 Wire Wire Line
 	3200 5400 3200 5450
@@
 	3200 5450 3200 5500
 $Comp
-L Asiste:GND #PWR0304
+L Asiste:GND #PWR015
 U 1 1 5B744A7C
 P 3900 3550
-F 0 "#PWR0304" H 3900 3300 50  0001 C CNN
+F 0 "#PWR015" H 3900 3300 50  0001 C CNN
 F 1 "GND" H 3905 3377 50  0000 C CNN
 F 2 "" H 3900 3550 50  0001 C CNN
@@
 	3900 2550 3900 2600
 $Comp
-L Asiste:VBAT #PWR0305
+L Asiste:VBAT #PWR016
 U 1 1 5B7453C9
 P 5300 2600
-F 0 "#PWR0305" H 5300 2450 50  0001 C CNN
+F 0 "#PWR016" H 5300 2450 50  0001 C CNN
 F 1 "VBAT" H 5315 2773 50  0000 C CNN
 F 2 "" H 5300 2600 50  0001 C CNN
@@
 	3900 3500 3900 3550
 $Comp
-L Asiste:C_0603_4.7uF C301
+L Asiste:C_0603_4.7uF C4
 U 1 1 5B745D35
 P 2650 3050
-F 0 "C301" H 2536 3004 50  0000 R CNN
+F 0 "C4" H 2536 3004 50  0000 R CNN
 F 1 "C_0603_4.7uF" H 2450 2500 50  0001 L CNN
 F 2 "ASISTE:C_0603" H 2700 2800 50  0001 C CNN
@@
 Connection ~ 3300 3500
 $Comp
-L Asiste:C_0603_4.7uF C302
+L Asiste:C_0603_4.7uF C5
 U 1 1 5B74635C
 P 5300 3050
-F 0 "C302" H 5415 3096 50  0000 L CNN
+F 0 "C5" H 5415 3096 50  0000 L CNN
 F 1 "C_0603_4.7uF" H 5100 2500 50  0001 L CNN
 F 2 "ASISTE:C_0603" H 5350 2800 50  0001 C CNN
@@
 	4300 3100 4400 3100
 $Comp
-L Asiste:R_0402_2k R301
+L Asiste:R_0402_2k R8
 U 1 1 5B74B4B5
 P 3300 3300
-F 0 "R301" H 3370 3346 50  0000 L CNN
+F 0 "R8" H 3370 3346 50  0000 L CNN
 F 1 "R_0402_2k" H 3300 2750 50  0001 C CNN
 F 2 "ASISTE:R_0402" H 3300 2850 50  0001 C CNN
@@
 $EndComp
 $Comp
-L Asiste:R_0402_2M2 R303
+L Asiste:R_0402_2M2 R10
 U 1 1 5B74D1E7
 P 5900 3250
-F 0 "R303" H 5970 3296 50  0000 L CNN
+F 0 "R10" H 5970 3296 50  0000 L CNN
 F 1 "R_0402_2M2" H 5900 2700 50  0001 C CNN
 F 2 "ASISTE:R_0402" H 5900 2800 50  0001 C CNN
@@
 $EndComp
 $Comp
-L Asiste:R_0402_10M R302
+L Asiste:R_0402_10M R9
 U 1 1 5B74D9F6
 P 5900 2850
-F 0 "R302" H 5970 2896 50  0000 L CNN
+F 0 "R9" H 5970 2896 50  0000 L CNN
 F 1 "R_0402_10M" H 5900 2300 50  0001 C CNN
 F 2 "ASISTE:R_0402" H 5900 2400 50  0001 C CNN
@@
 BAT_SENSE
 $Comp
-L Asiste:VBUS #PWR0302
+L Asiste:VBUS #PWR013
 U 1 1 5B795544
 P 3600 4700
-F 0 "#PWR0302" H 3600 4550 50  0001 C CNN
+F 0 "#PWR013" H 3600 4550 50  0001 C CNN
 F 1 "VBUS" H 3615 4873 50  0000 C CNN
 F 2 "" H 3600 4700 50  0001 C CNN
@@
 $EndComp
 $Comp
-L Asiste:VBUS #PWR0303
+L Asiste:VBUS #PWR014
 U 1 1 5B7955CD
 P 3900 2550
-F 0 "#PWR0303" H 3900 2400 50  0001 C CNN
+F 0 "#PWR014" H 3900 2400 50  0001 C CNN
 F 1 "VBUS" H 3915 2723 50  0000 C CNN
 F 2 "" H 3900 2550 50  0001 C CNN
@@
 	2300 6900 1100 6900
 $Comp
-L Asiste:Conn_01x02 J302
+L Asiste:Conn_01x02 J2
 U 1 1 5B79A067
 P 7450 2600
-F 0 "J302" H 7530 2592 50  0000 L CNN
+F 0 "J2" H 7530 2592 50  0000 L CNN
 F 1 "Conn_01x02" H 7530 2501 50  0000 L CNN
 F 2 "ASISTE:JST_SH_SM02B-SRSS-TB_1x02-1MP_P1.00mm_Horizontal" H 7500 2100 50  0001 C CNN
@@
 Connection ~ 5900 3500
 $Comp
-L Asiste:DMP1045U Q301
+L Asiste:DMP1045U Q4
 U 1 1 5B86EC1C
 P 7950 1900
-F 0 "Q301" V 8200 1900 50  0000 C CNN
+F 0 "Q4" V 8200 1900 50  0000 C CNN
 F 1 "DMP1045U" V 8291 1900 50  0000 C CNN
 F 2 "ASISTE:SOT-23" H 8050 1400 50  0001 C CNN
@@
 	3150 2600 3900 2600
 $Comp
-L Asiste:D_Schottky D301
+L Asiste:D_Schottky D2
 U 1 1 5B8728BF
 P 8700 1750
-F 0 "D301" V 8746 1671 50  0000 R CNN
+F 0 "D2" V 8746 1671 50  0000 R CNN
 F 1 "D_Schottky" V 8655 1671 50  0000 R CNN
 F 2 "ASISTE:D_SOD-123" H 8700 1350 50  0001 C CNN
@@
 	8700 2000 8700 1900
 $Comp
-L Asiste:C_0603_1uF C306
+L Asiste:C_0603_1uF C9
 U 1 1 5B875437
 P 8700 3050
-F 0 "C306" H 8815 3096 50  0000 L CNN
+F 0 "C9" H 8815 3096 50  0000 L CNN
 F 1 "C_0603_1uF" H 8500 2500 50  0001 L CNN
 F 2 "ASISTE:C_0603" H 8750 2800 50  0001 C CNN
@@
 Connection ~ 7250 3500
 $Comp
-L Asiste:R_0402_100k R304
+L Asiste:R_0402_100k R11
 U 1 1 5B87AE63
 P 9500 2500
-F 0 "R304" H 9570 2546 50  0000 L CNN
+F 0 "R11" H 9570 2546 50  0000 L CNN
 F 1 "R_0402_100k" H 9500 1950 50  0001 C CNN
 F 2 "ASISTE:R_0402" H 9500 2050 50  0001 C CNN
@@
 Connection ~ 8700 3500
 $Comp
-L Asiste:VCC #PWR0310
+L Asiste:VCC #PWR021
 U 1 1 5B882208
 P 8800 2000
-F 0 "#PWR0310" H 8800 1850 50  0001 C CNN
+F 0 "#PWR021" H 8800 1850 50  0001 C CNN
 F 1 "VCC" V 8815 2128 50  0000 L CNN
 F 2 "" H 8800 2000 50  0001 C CNN
@@
 	8700 2000 8800 2000
 $Comp
-L Asiste:XC6415CC91MR-G U302
+L Asiste:XC6415CC91MR-G U2
 U 1 1 5B890199
 P 7350 5000
-F 0 "U302" H 7050 5200 60  0000 C CNN
+F 0 "U2" H 7050 5200 60  0000 C CNN
 F 1 "XC6415CC91MR-G" H 7850 5200 60  0000 C CNN
 F 2 "ASISTE:TSOT-23-6" H 6950 5100 60  0001 C CNN
@@
 $EndComp
 $Comp
-L Asiste:VCC #PWR0306
+L Asiste:VCC #PWR017
 U 1 1 5B890448
 P 7350 4600
-F 0 "#PWR0306" H 7350 4450 50  0001 C CNN
+F 0 "#PWR017" H 7350 4450 50  0001 C CNN
 F 1 "VCC" H 7365 4773 50  0000 C CNN
 F 2 "" H 7350 4600 50  0001 C CNN
@@
 	7350 4600 7350 4650
 $Comp
-L Asiste:GND #PWR0307
+L Asiste:GND #PWR018
 U 1 1 5B8910DA
 P 7350 5750
-F 0 "#PWR0307" H 7350 5500 50  0001 C CNN
+F 0 "#PWR018" H 7350 5500 50  0001 C CNN
 F 1 "GND" H 7355 5577 50  0000 C CNN
 F 2 "" H 7350 5750 50  0001 C CNN
@@
 Wire Wire Line
 	7350 4650 7350 4750
-Text HLabel 6500 4950 0    60   Input ~ 0
-PWR_EN
-Wire Wire Line
-	6500 4950 6900 4950
 Wire Wire Line
 	8500 4950 8500 4850
@@
 	7800 4950 8500 4950
 $Comp
-L Asiste:C_0603_1uF C305
+L Asiste:C_0603_1uF C8
 U 1 1 5B89B89A
 P 8500 5450
-F 0 "C305" H 8615 5496 50  0000 L CNN
+F 0 "C8" H 8615 5496 50  0000 L CNN
 F 1 "C_0603_1uF" H 8300 4900 50  0001 L CNN
 F 2 "ASISTE:C_0603" H 8550 5200 50  0001 C CNN
@@
 $EndComp
 $Comp
-L Asiste:C_0603_1uF C304
+L Asiste:C_0603_1uF C7
 U 1 1 5B89B95E
 P 7950 5450
-F 0 "C304" H 8065 5496 50  0000 L CNN
+F 0 "C7" H 8065 5496 50  0000 L CNN
 F 1 "C_0603_1uF" H 7750 4900 50  0001 L CNN
 F 2 "ASISTE:C_0603" H 8000 5200 50  0001 C CNN
@@
 Connection ~ 8500 4950
 $Comp
-L Asiste:C_0603_1uF C303
+L Asiste:C_0603_1uF C6
 U 1 1 5B8A2E24
 P 6800 5450
-F 0 "C303" H 6915 5496 50  0000 L CNN
+F 0 "C6" H 6915 5496 50  0000 L CNN
 F 1 "C_0603_1uF" H 6600 4900 50  0001 L CNN
 F 2 "ASISTE:C_0603" H 6850 5200 50  0001 C CNN
@@
 	6800 5700 7350 5700
 $Comp
-L Asiste:+1V8 #PWR0309
+L Asiste:+1V8 #PWR020
 U 1 1 5B8AB235
 P 8500 4850
-F 0 "#PWR0309" H 8500 4700 50  0001 C CNN
+F 0 "#PWR020" H 8500 4700 50  0001 C CNN
 F 1 "+1V8" H 8650 4900 50  0000 C CNN
 F 2 "" H 8500 4850 50  0001 C CNN
@@
 $EndComp
 $Comp
-L Asiste:+3V3 #PWR0308
+L Asiste:+3V3 #PWR019
 U 1 1 5B8AB308
 P 7950 5150
-F 0 "#PWR0308" H 7950 5000 50  0001 C CNN
+F 0 "#PWR019" H 7950 5000 50  0001 C CNN
 F 1 "+3V3" H 8100 5200 50  0000 C CNN
 F 2 "" H 7950 5150 50  0001 C CNN
@@
 $EndComp
 Wire Wire Line
-	6800 4650 6800 5200
-$Comp
-L Asiste:PWR_FLAG #FLG0301
+	6800 4650 6800 4950
+$Comp
+L Asiste:PWR_FLAG #FLG01
 U 1 1 5B8BB2C5
 P 7650 4600
-F 0 "#FLG0301" H 7650 4675 50  0001 C CNN
+F 0 "#FLG01" H 7650 4675 50  0001 C CNN
 F 1 "PWR_FLAG" H 7650 4774 50  0000 C CNN
 F 2 "" H 7650 4600 50  0001 C CNN
@@
 	4550 2600 4550 2900
 $Comp
-L Asiste:MCP73831 U301
+L Asiste:MCP73831 U1
 U 1 1 5B8C4CF4
 P 3900 3000
-F 0 "U301" H 3650 3250 50  0000 C CNN
+F 0 "U1" H 3650 3250 50  0000 C CNN
 F 1 "MCP73831" H 4150 3250 50  0000 C CNN
 F 2 "ASISTE:TSOT-23-5" H 3400 2250 50  0001 L CIN
@@
 	1    0    0    -1
 $EndComp
+$Comp
+L Asiste:USB_B_Micro_SMD J1
+U 1 1 5B957D61
+P 3200 5000
+F 0 "J1" H 3050 5350 50  0000 C CNN
+F 1 "USB_B_Micro_SMD" V 2950 5050 50  0001 C CNN
+F 2 "ASISTE:USB_Micro-B_Molex_47346-0001" H 3150 4250 50  0001 C CNN
+F 3 "https://www.mouser.es/datasheet/2/276/0473460001_IO_CONNECTORS-229243.pdf" H 3250 4150 50  0001 C CNN
+F 4 "47346-0001" H 3200 4050 60  0001 C CNN "man#"
+	1    3200 5000
+	1    0    0    -1
+$EndComp
+Wire Wire Line
+	6900 4950 6800 4950
+Connection ~ 6800 4950
+Wire Wire Line
+	6800 4950 6800 5200
 $EndSCHEMATC

Commit message: Actualizando
Parts:
- R8: Resistance 2k -> 10k
- U2: man# XC6415CC91MR-G -> XC6415CC06MR-G
- renumbered C4 to C3, C5 to C4, C6 to C5, C7 to C6, C8 to C7, C9 to C8
Other:
- note removed: "IREG= 1000V/RPROG\nRPROG = kOhms\nIREG = miliampere"
