File: temperature.sch (KiCad schematic (older format))
At the start: 5 parts

Commit message: Esquemático parcialmente revisado. Falta revisar pines y correspondencia con footprints
Parts:
- gave numbers to parts that had none: 5
Connections:
- wire segments 24 -> 25
Changed lines of the file:
@@
 $Descr A4 11693 8268
 encoding utf-8
-Sheet 6 6
+Sheet 5 6
 Title "Temperature"
 Date "2018-08-15"
@@
 $EndDescr
 $Comp
-L Asiste:TMP112AIDRLR U?
+L Asiste:TMP112AIDRLR U601
 U 1 1 5B7E0916
 P 5900 3850
-F 0 "U?" H 5600 4200 60  0000 L CNN
+F 0 "U601" H 5600 4200 60  0000 L CNN
 F 1 "TMP112AIDRLR" H 4900 3700 60  0000 L CNN
 F 2 "ASISTE:SOT-563" H 6100 4050 60  0001 L CNN
@@
 $EndComp
 $Comp
-L Asiste:R_0402_10k R?
+L Asiste:R_0402_10k R602
 U 1 1 5B7E0A13
 P 5150 3400
-F 0 "R?" H 5220 3446 50  0000 L CNN
+F 0 "R602" H 5220 3446 50  0000 L CNN
 F 1 "R_0402_10k" H 5150 2850 50  0001 C CNN
 F 2 "ASISTE:R_0402" H 5150 2950 50  0001 C CNN
@@
 $EndComp
 $Comp
-L Asiste:R_0402_10k R?
+L Asiste:R_0402_10k R601
 U 1 1 5B7E0A91
 P 4850 3400
-F 0 "R?" H 4780 3354 50  0000 R CNN
+F 0 "R601" H 4780 3354 50  0000 R CNN
 F 1 "R_0402_10k" H 4850 2850 50  0001 C CNN
 F 2 "ASISTE:R_0402" H 4850 2950 50  0001 C CNN
@@
 $EndComp
 $Comp
-L Asiste:+3V3 #PWR?
+L Asiste:+3V3 #PWR0601
 U 1 1 5B7E0B01
 P 5000 3150
-F 0 "#PWR?" H 5000 3000 50  0001 C CNN
+F 0 "#PWR0601" H 5000 3000 50  0001 C CNN
 F 1 "+3V3" H 5015 3323 50  0000 C CNN
 F 2 "" H 5000 3150 50  0001 C CNN
@@
 TMP_SDA
 $Comp
-L Asiste:R_0402_10k R?
+L Asiste:R_0402_10k R603
 U 1 1 5B7E0E26
 P 6600 3600
-F 0 "R?" H 6670 3646 50  0000 L CNN
+F 0 "R603" H 6670 3646 50  0000 L CNN
 F 1 "R_0402_10k" H 6600 3050 50  0001 C CNN
 F 2 "ASISTE:R_0402" H 6600 3150 50  0001 C CNN
@@
 TMP_ALERT
 $Comp
-L Asiste:GND #PWR?
+L Asiste:GND #PWR0602
 U 1 1 5B7E103E
 P 5800 4400
-F 0 "#PWR?" H 5800 4150 50  0001 C CNN
+F 0 "#PWR0602" H 5800 4150 50  0001 C CNN
 F 1 "GND" H 5805 4227 50  0000 C CNN
 F 2 "" H 5800 4400 50  0001 C CNN
@@
 	6600 3250 6600 3450
 $Comp
-L Asiste:+3V3 #PWR?
+L Asiste:+3V3 #PWR0604
 U 1 1 5B7E1276
 P 6300 3200
-F 0 "#PWR?" H 6300 3050 50  0001 C CNN
+F 0 "#PWR0604" H 6300 3050 50  0001 C CNN
 F 1 "+3V3" H 6315 3373 50  0000 C CNN
 F 2 "" H 6300 3200 50  0001 C CNN
@@
 	6300 3200 6300 3250
 $Comp
-L Asiste:C_0402_100nF C?
+L Asiste:C_0402_100nF C601
 U 1 1 5B7E174A
 P 6300 4100
-F 0 "C?" H 6415 4146 50  0000 L CNN
+F 0 "C601" H 6415 4146 50  0000 L CNN
 F 1 "C_0402_100nF" H 6050 3550 50  0001 L CNN
 F 2 "ASISTE:C_0402" H 6350 3850 50  0001 C CNN
@@
 Wire Wire Line
 	6200 3850 6600 3850
+$Comp
+L Asiste:GND #PWR0603
+U 1 1 5B8BAB14
+P 5900 3350
+F 0 "#PWR0603" H 5900 3100 50  0001 C CNN
+F 1 "GND" H 5905 3177 50  0000 C CNN
+F 2 "" H 5900 3350 50  0001 C CNN
+F 3 "" H 5900 3350 50  0001 C CNN
+	1    5900 3350
+	-1   0    0    1
+$EndComp
+Wire Wire Line
+	5900 3350 5900 3450
 $EndSCHEMATC

Commit message: Añadido botón y otros
Parts:
- renumbered C601 to C501, R601 to R501, R602 to R502, R603 to R503, U601 to U501
Changed lines of the file:
@@
 $EndDescr
 $Comp
-L Asiste:TMP112AIDRLR U601
+L Asiste:TMP112AIDRLR U501
 U 1 1 5B7E0916
 P 5900 3850
-F 0 "U601" H 5600 4200 60  0000 L CNN
+F 0 "U501" H 5600 4200 60  0000 L CNN
 F 1 "TMP112AIDRLR" H 4900 3700 60  0000 L CNN
 F 2 "ASISTE:SOT-563" H 6100 4050 60  0001 L CNN
@@
 $EndComp
 $Comp
-L Asiste:R_0402_10k R602
+L Asiste:R_0402_10k R502
 U 1 1 5B7E0A13
 P 5150 3400
-F 0 "R602" H 5220 3446 50  0000 L CNN
+F 0 "R502" H 5220 3446 50  0000 L CNN
 F 1 "R_0402_10k" H 5150 2850 50  0001 C CNN
 F 2 "ASISTE:R_0402" H 5150 2950 50  0001 C CNN
@@
 $EndComp
 $Comp
-L Asiste:R_0402_10k R601
+L Asiste:R_0402_10k R501
 U 1 1 5B7E0A91
 P 4850 3400
-F 0 "R601" H 4780 3354 50  0000 R CNN
+F 0 "R501" H 4780 3354 50  0000 R CNN
 F 1 "R_0402_10k" H 4850 2850 50  0001 C CNN
 F 2 "ASISTE:R_0402" H 4850 2950 50  0001 C CNN
@@
 $EndComp
 $Comp
-L Asiste:+3V3 #PWR0601
+L Asiste:+3V3 #PWR0501
 U 1 1 5B7E0B01
 P 5000 3150
-F 0 "#PWR0601" H 5000 3000 50  0001 C CNN
+F 0 "#PWR0501" H 5000 3000 50  0001 C CNN
 F 1 "+3V3" H 5015 3323 50  0000 C CNN
 F 2 "" H 5000 3150 50  0001 C CNN
@@
 TMP_SDA
 $Comp
-L Asiste:R_0402_10k R603
+L Asiste:R_0402_10k R503
 U 1 1 5B7E0E26
 P 6600 3600
-F 0 "R603" H 6670 3646 50  0000 L CNN
+F 0 "R503" H 6670 3646 50  0000 L CNN
 F 1 "R_0402_10k" H 6600 3050 50  0001 C CNN
 F 2 "ASISTE:R_0402" H 6600 3150 50  0001 C CNN
@@
 TMP_ALERT
 $Comp
-L Asiste:GND #PWR0602
+L Asiste:GND #PWR0502
 U 1 1 5B7E103E
 P 5800 4400
-F 0 "#PWR0602" H 5800 4150 50  0001 C CNN
+F 0 "#PWR0502" H 5800 4150 50  0001 C CNN
 F 1 "GND" H 5805 4227 50  0000 C CNN
 F 2 "" H 5800 4400 50  0001 C CNN
@@
 	6600 3250 6600 3450
 $Comp
-L Asiste:+3V3 #PWR0604
+L Asiste:+3V3 #PWR0504
 U 1 1 5B7E1276
 P 6300 3200
-F 0 "#PWR0604" H 6300 3050 50  0001 C CNN
+F 0 "#PWR0504" H 6300 3050 50  0001 C CNN
 F 1 "+3V3" H 6315 3373 50  0000 C CNN
 F 2 "" H 6300 3200 50  0001 C CNN
@@
 	6300 3200 6300 3250
 $Comp
-L Asiste:C_0402_100nF C601
+L Asiste:C_0402_100nF C501
 U 1 1 5B7E174A
 P 6300 4100
-F 0 "C601" H 6415 4146 50  0000 L CNN
+F 0 "C501" H 6415 4146 50  0000 L CNN
 F 1 "C_0402_100nF" H 6050 3550 50  0001 L CNN
 F 2 "ASISTE:C_0402" H 6350 3850 50  0001 C CNN
@@
 	6200 3850 6600 3850
 $Comp
-L Asiste:GND #PWR0603
+L Asiste:GND #PWR0503
 U 1 1 5B8BAB14
 P 5900 3350
-F 0 "#PWR0603" H 5900 3100 50  0001 C CNN
+F 0 "#PWR0503" H 5900 3100 50  0001 C CNN
 F 1 "GND" H 5905 3177 50  0000 C CNN
 F 2 "" H 5900 3350 50  0001 C CNN

Commit message: Esquemáticos totalmente terminados y revisados PCB a falta de routear el puerto de programación
Parts:
- removed R501, R502, R503: R_0402_10k, ASISTE:R_0402, symbol Asiste:R_0402_10k
- added R15: R_0402_4k7, ASISTE:R_0402, symbol Asiste:R_0402_4k7
- renumbered C501 to C14, U501 to U4
Connections:
- wire segments 25 -> 13
Changed lines of the file:
@@
 $EndDescr
 $Comp
-L Asiste:TMP112AIDRLR U501
+L Asiste:TMP112AIDRLR U4
 U 1 1 5B7E0916
 P 5900 3850
-F 0 "U501" H 5600 4200 60  0000 L CNN
+F 0 "U4" H 5600 4200 60  0000 L CNN
 F 1 "TMP112AIDRLR" H 4900 3700 60  0000 L CNN
 F 2 "ASISTE:SOT-563" H 6100 4050 60  0001 L CNN
@@
 	1    0    0    -1
 $EndComp
-$Comp
-L Asiste:R_0402_10k R502
-U 1 1 5B7E0A13
-P 5150 3400
-F 0 "R502" H 5220 3446 50  0000 L CNN
-F 1 "R_0402_10k" H 5150 2850 50  0001 C CNN
-F 2 "ASISTE:R_0402" H 5150 2950 50  0001 C CNN
-F 3 "https://www.mouser.es/datasheet/2/315/AOA0000C334-1314047.pdf" H 5150 3050 50  0001 C CNN
-F 4 "ERJ-U02D1002X" H 5100 3150 60  0001 C CNN "man#"
-F 5 "10k" H 5220 3355 50  0000 L CNN "Resistance"
-	1    5150 3400
-	1    0    0    -1
-$EndComp
-$Comp
-L Asiste:R_0402_10k R501
-U 1 1 5B7E0A91
-P 4850 3400
-F 0 "R501" H 4780 3354 50  0000 R CNN
-F 1 "R_0402_10k" H 4850 2850 50  0001 C CNN
-F 2 "ASISTE:R_0402" H 4850 2950 50  0001 C CNN
-F 3 "https://www.mouser.es/datasheet/2/315/AOA0000C334-1314047.pdf" H 4850 3050 50  0001 C CNN
-F 4 "ERJ-U02D1002X" H 4800 3150 60  0001 C CNN "man#"
-F 5 "10k" H 4780 3445 50  0000 R CNN "Resistance"
-	1    4850 3400
-	1    0    0    1
-$EndComp
-$Comp
-L Asiste:+3V3 #PWR0501
-U 1 1 5B7E0B01
-P 5000 3150
-F 0 "#PWR0501" H 5000 3000 50  0001 C CNN
-F 1 "+3V3" H 5015 3323 50  0000 C CNN
-F 2 "" H 5000 3150 50  0001 C CNN
-F 3 "" H 5000 3150 50  0001 C CNN
-	1    5000 3150
-	1    0    0    -1
-$EndComp
-Wire Wire Line
-	4850 3250 4850 3200
-Wire Wire Line
-	4850 3200 5000 3200
-Wire Wire Line
-	5150 3200 5150 3250
-Wire Wire Line
-	5000 3150 5000 3200
-Connection ~ 5000 3200
-Wire Wire Line
-	5000 3200 5150 3200
-Wire Wire Line
-	5150 3550 5150 3650
-Wire Wire Line
-	5150 3650 5500 3650
-Wire Wire Line
-	4850 3550 4850 3750
-Wire Wire Line
-	4850 3750 5500 3750
-Wire Wire Line
-	5150 3650 4450 3650
-Connection ~ 5150 3650
-Wire Wire Line
-	4850 3750 4450 3750
-Connection ~ 4850 3750
 Text HLabel 4450 3650 0    60   Input ~ 0
 TMP_SCL
 Text HLabel 4450 3750 0    60   BiDi ~ 0
 TMP_SDA
-$Comp
-L Asiste:R_0402_10k R503
-U 1 1 5B7E0E26
-P 6600 3600
-F 0 "R503" H 6670 3646 50  0000 L CNN
-F 1 "R_0402_10k" H 6600 3050 50  0001 C CNN
-F 2 "ASISTE:R_0402" H 6600 3150 50  0001 C CNN
-F 3 "https://www.mouser.es/datasheet/2/315/AOA0000C334-1314047.pdf" H 6600 3250 50  0001 C CNN
-F 4 "ERJ-U02D1002X" H 6550 3350 60  0001 C CNN "man#"
-F 5 "10k" H 6670 3555 50  0000 L CNN "Resistance"
-	1    6600 3600
-	1    0    0    -1
-$EndComp
-Wire Wire Line
-	6600 3850 6600 3750
 Text HLabel 6850 3850 2    60   Output ~ 0
 TMP_ALERT
 $Comp
-L Asiste:GND #PWR0502
+L Asiste:GND #PWR028
 U 1 1 5B7E103E
 P 5800 4400
-F 0 "#PWR0502" H 5800 4150 50  0001 C CNN
+F 0 "#PWR028" H 5800 4150 50  0001 C CNN
 F 1 "GND" H 5805 4227 50  0000 C CNN
 F 2 "" H 5800 4400 50  0001 C CNN
@@
 Wire Wire Line
 	6000 3450 6000 3250
-Wire Wire Line
-	6600 3250 6600 3450
 $Comp
-L Asiste:+3V3 #PWR0504
+L Asiste:+3V3 #PWR030
 U 1 1 5B7E1276
-P 6300 3200
-F 0 "#PWR0504" H 6300 3050 50  0001 C CNN
-F 1 "+3V3" H 6315 3373 50  0000 C CNN
-F 2 "" H 6300 3200 50  0001 C CNN
-F 3 "" H 6300 3200 50  0001 C CNN
-	1    6300 3200
+P 6300 2750
+F 0 "#PWR030" H 6300 2600 50  0001 C CNN
+F 1 "+3V3" H 6315 2923 50  0000 C CNN
+F 2 "" H 6300 2750 50  0001 C CNN
+F 3 "" H 6300 2750 50  0001 C CNN
+	1    6300 2750
 	1    0    0    -1
 $EndComp
-Wire Wire Line
-	6300 3200 6300 3250
 $Comp
-L Asiste:C_0402_100nF C501
+L Asiste:C_0402_100nF C14
 U 1 1 5B7E174A
 P 6300 4100
-F 0 "C501" H 6415 4146 50  0000 L CNN
+F 0 "C14" H 6415 4146 50  0000 L CNN
 F 1 "C_0402_100nF" H 6050 3550 50  0001 L CNN
 F 2 "ASISTE:C_0402" H 6350 3850 50  0001 C CNN
@@
 	6000 3250 6300 3250
 Connection ~ 6300 3250
-Wire Wire Line
-	6300 3250 6600 3250
-Connection ~ 6600 3850
-Wire Wire Line
-	6600 3850 6850 3850
-Wire Wire Line
-	6200 3850 6600 3850
 $Comp
-L Asiste:GND #PWR0503
+L Asiste:GND #PWR029
 U 1 1 5B8BAB14
 P 5900 3350
-F 0 "#PWR0503" H 5900 3100 50  0001 C CNN
+F 0 "#PWR029" H 5900 3100 50  0001 C CNN
 F 1 "GND" H 5905 3177 50  0000 C CNN
 F 2 "" H 5900 3350 50  0001 C CNN
@@
 Wire Wire Line
 	5900 3350 5900 3450
+Wire Wire Line
+	6300 3150 6300 3250
+Wire Wire Line
+	6300 2750 6300 2850
+Wire Wire Line
+	4450 3650 5500 3650
+Wire Wire Line
+	4450 3750 5500 3750
+Wire Wire Line
+	6200 3850 6850 3850
+$Comp
+L Asiste:R_0402_4k7 R15
+U 1 1 5B99BD78
+P 6300 3000
+F 0 "R15" H 6400 3050 50  0000 L CNN
+F 1 "R_0402_4k7" H 6300 2450 50  0001 C CNN
+F 2 "ASISTE:R_0402" H 6300 2550 50  0001 C CNN
+F 3 "https://www.mouser.es/datasheet/2/315/AOA0000C334-1314047.pdf" H 6300 2650 50  0001 C CNN
+F 4 "ERJ-U02D4701X" H 6250 2750 60  0001 C CNN "man#"
+F 5 "4k7" H 6400 2950 50  0000 L CNN "Resistance"
+	1    6300 3000
+	1    0    0    -1
+$EndComp
 $EndSCHEMATC

Commit message: Actualizando
Parts:
- renumbered C14 to C13
Changed lines of the file:
@@
 $EndComp
 $Comp
-L Asiste:C_0402_100nF C14
+L Asiste:C_0402_100nF C13
 U 1 1 5B7E174A
 P 6300 4100
-F 0 "C14" H 6415 4146 50  0000 L CNN
+F 0 "C13" H 6415 4146 50  0000 L CNN
 F 1 "C_0402_100nF" H 6050 3550 50  0001 L CNN
 F 2 "ASISTE:C_0402" H 6350 3850 50  0001 C CNN
